File: Project QUBO/eagleDesigns/powerBoard/Power Supply Board.brd (EAGLE design)
At the start: 101.6 x 101.6 mm, 87 parts

Commit message: updated psb sch
Parts:
- removed CURRENTSENSOR12, CURRENTSENSOR3.3, CURRENTSENSOR5: ACS764, allegro:ACS764
- removed R10, R13, R7: 10 kΩ, resistor:R0603
- removed R11, R12, R14, R15, R8, R9: 107 kΩ, resistor:R0603
- added C24, C25, C26, C27: 2.2 µF, resistor:C1206
- added C28: 100 nF, resistor:C0603
- added C29: 10 µF, resistor:C0805
- added C30: 100 uF, resistor:PANASONIC_D
- added R22: 732 Ω, resistor:R0603
- added REG-9V: PTN78060W, texas:PTN78060W
- R3: value 732 Ω -> 407 kΩ
- moved REG-12V 331.8 mm to (-110.5, -510.5)
Connections:
- removed net I2C-SDA: CURRENTSENSOR12.P$15, CURRENTSENSOR3.3.P$15, CURRENTSENSOR5.P$15
- removed net I2C-SDL: CURRENTSENSOR12.P$16, CURRENTSENSOR3.3.P$16, CURRENTSENSOR5.P$16
- removed net N$18: CURRENTSENSOR5.P$18
- removed net N$19: CURRENTSENSOR3.3.P$18
- removed net N$20: CURRENTSENSOR5.P$4, R10.2
- removed net N$21: CURRENTSENSOR5.P$5
- removed net N$22: CURRENTSENSOR5.P$6
- removed net N$23: CURRENTSENSOR3.3.P$4, R7.2
- removed net N$24: CURRENTSENSOR3.3.P$5
- removed net N$25: CURRENTSENSOR3.3.P$6
- removed net N$28: CURRENTSENSOR12.P$18
- removed net N$29: CURRENTSENSOR12.P$4, R13.2
- removed net N$30: CURRENTSENSOR12.P$5
- removed net N$31: CURRENTSENSOR12.P$6
- new net N$37: R22.2, REG-12V.P$6
- net 12VACS: now also C28.1, C29.1, C30.+, REG-9V.P$5, REG-9V.P$7
- net 3.3V: no longer CURRENTSENSOR12.P$1, CURRENTSENSOR12.P$10, CURRENTSENSOR12.P$11, CURRENTSENSOR12.P$12, CURRENTSENSOR12.P$14, CURRENTSENSOR12.P$2, CURRENTSENSOR12.P$7, CURRENTSENSOR12.P$8, CURRENTSENSOR12.P$9, CURRENTSENSOR3.3.P$1, CURRENTSENSOR3.3.P$10, CURRENTSENSOR3.3.P$11, CURRENTSENSOR3.3.P$12, CURRENTSENSOR3.3.P$14, CURRENTSENSOR3.3.P$7, CURRENTSENSOR3.3.P$8, CURRENTSENSOR3.3.P$9, CURRENTSENSOR5.P$1, CURRENTSENSOR5.P$10, CURRENTSENSOR5.P$11, CURRENTSENSOR5.P$12, CURRENTSENSOR5.P$14, CURRENTSENSOR5.P$3, CURRENTSENSOR5.P$7, CURRENTSENSOR5.P$8, CURRENTSENSOR5.P$9, R10.1, R11.1, R12.1, R13.1, R14.1, R15.1, R7.1, R8.1, R9.1
- net 3.3VACS: no longer CURRENTSENSOR12.P$13, CURRENTSENSOR12.P$19, CURRENTSENSOR12.P$20, CURRENTSENSOR12.P$21, CURRENTSENSOR12.P$22, CURRENTSENSOR12.P$23, CURRENTSENSOR12.P$24, CURRENTSENSOR3.3.P$13, CURRENTSENSOR3.3.P$19, CURRENTSENSOR3.3.P$20, CURRENTSENSOR3.3.P$21, CURRENTSENSOR3.3.P$22, CURRENTSENSOR3.3.P$23, CURRENTSENSOR3.3.P$24, CURRENTSENSOR5.P$13, CURRENTSENSOR5.P$19, CURRENTSENSOR5.P$20, CURRENTSENSOR5.P$21, CURRENTSENSOR5.P$22, CURRENTSENSOR5.P$23, CURRENTSENSOR5.P$24
- net GND: now also C24.2, C25.2, C26.2, C27.2, C28.2, C29.2, C30.-, R22.1, REG-9V.P$1, REG-9V.P$2; no longer CURRENTSENSOR12.P$17, CURRENTSENSOR12.P$3, CURRENTSENSOR3.3.P$17, CURRENTSENSOR3.3.P$2, CURRENTSENSOR3.3.P$3, CURRENTSENSOR5.P$17, CURRENTSENSOR5.P$2, R11.2, R12.2, R14.2, R15.2, R8.2, R9.2
- net N$4: now also REG-9V.P$6; no longer REG-12V.P$6
- net VI12V: now also C24.1, C25.1, C26.1, C27.1, REG-9V.P$4

Commit message: edited power supply board sch
Parts:
- removed UVQ: UVQ-24/4.5-D24P-C, murata:UVQ-24/4.5-D24P-C
- added U$3: UWEUWE, murata:UWE
Connections:
- new net UVQ+: U$3.+SENSE, U$3.+VOUT
- new net UVQ-: U$3.-SENSE, U$3.-VOUT
- net UVQV+: no longer UVQ.P$8
- net UVQV-: no longer UVQ.P$4
Changed lines of the file:
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@@
 <element name="HOTSWAP1" library="linear" package="LTC4231" value="LTC4231" x="-52.07" y="81.28"/>
 <element name="BAT2-CON" library="molex" package="172043-0201" value="172043-0201" x="54.61" y="7.62" rot="R180"/>
-<element name="UVQ" library="murata" package="UVQ-24/4.5-D24P-C" value="UVQ-24/4.5-D24P-C" x="31.75" y="40.64"/>
 <element name="U$18" library="texas" package="CSD19537Q3" value="CSD19537Q3" x="-88.9" y="2.54"/>
 <element name="REG-3.3V" library="texas" package="PTN78060W" value="PTN78060W" x="-95.25" y="-8.89"/>
@@
 <element name="C29" library="resistor" package="C0805" value="10 µF" x="-106.68" y="-529.59"/>
 <element name="C30" library="resistor" package="PANASONIC_D" value="100 uF" x="-119.38" y="-523.24"/>
+<element name="U$3" library="murata" package="UWE" value="UWEUWE" x="-93.98" y="-551.18"/>
 </elements>
 <signals>
@@
 <signal name="UVQV+">
 <contactref element="U$14" pad="CKT1"/>
-<contactref element="UVQ" pad="P$8"/>
-<wire x1="57.15" y1="33.02" x2="72.62" y2="9.1" width="0" layer="19" extent="1-1"/>
 </signal>
 <signal name="UVQV-">
 <contactref element="U$14" pad="CKT2"/>
-<contactref element="UVQ" pad="P$4"/>
-<wire x1="57.15" y1="48.26" x2="69.62" y2="9.1" width="0" layer="19" extent="1-1"/>
 </signal>
 <signal name="N$3">
@@
 <wire x1="-99.3775" y1="-516.89" x2="-99.48" y2="-529.59" width="0" layer="19" extent="1-1"/>
 </signal>
+<signal name="UVQ-">
+<contactref element="U$3" pad="-VOUT"/>
+<contactref element="U$3" pad="-SENSE"/>
+<wire x1="-68.58" y1="-543.56" x2="-68.58" y2="-547.37" width="0" layer="19" extent="1-1"/>
+</signal>
+<signal name="UVQ+">
+<contactref element="U$3" pad="+SENSE"/>
+<contactref element="U$3" pad="+VOUT"/>
+<wire x1="-68.58" y1="-554.99" x2="-68.58" y2="-558.8" width="0" layer="19" extent="1-1"/>
+</signal>
 </signals>
