File: Project QUBO/eagleDesigns/powerBoard/Power Supply Board.sch (EAGLE design)
At the start: 87 parts

Commit message: updated psb sch
Parts:
- removed CURRENTSENSOR12, CURRENTSENSOR3.3, CURRENTSENSOR5: ACS764, allegro:ACS764
- removed R10, R13, R7: 10 kΩ, resistor:R-US_R0603
- removed R11, R12, R14, R15, R8, R9: 107 kΩ, resistor:R-US_R0603
- added C24, C25, C26, C27: 2.2 µF, resistor:C-USC1206
- added C28: 100 nF, resistor:C-USC0603
- added C29: 10 µF, resistor:C-USC0805
- added C30: 100 uF, resistor:CPOL-USD
- added R22: 732 Ω, resistor:R-US_R0603
- added REG-9V: PTN78060W, texas:PTN78060W
- R3: value 732 Ω -> 407 kΩ
Connections:
- removed net I2C-SDA: CURRENTSENSOR12.SDA, CURRENTSENSOR3.3.SDA, CURRENTSENSOR5.SDA
- removed net I2C-SDL: CURRENTSENSOR12.SCL, CURRENTSENSOR3.3.SCL, CURRENTSENSOR5.SCL
- removed net N$18: CURRENTSENSOR5.NC
- removed net N$19: CURRENTSENSOR3.3.NC
- removed net N$20: CURRENTSENSOR5.FAULT, R10.2
- removed net N$21: CURRENTSENSOR5.FREEZE
- removed net N$22: CURRENTSENSOR5.NC2
- removed net N$23: CURRENTSENSOR3.3.FAULT, R7.2
- removed net N$24: CURRENTSENSOR3.3.FREEZE
- removed net N$25: CURRENTSENSOR3.3.NC2
- removed net N$28: CURRENTSENSOR12.NC
- removed net N$29: CURRENTSENSOR12.FAULT, R13.2
- removed net N$30: CURRENTSENSOR12.FREEZE
- removed net N$31: CURRENTSENSOR12.NC2
- new net N$37: R22.2, REG-12V.VOADJUST
- net 12VACS: now also C28.1, C29.1, C30.+, REG-9V.VO, REG-9V.VOSENSE
- net 3.3V: no longer CURRENTSENSOR12.A1, CURRENTSENSOR12.IP-, CURRENTSENSOR12.VCC, CURRENTSENSOR3.3.IP-, CURRENTSENSOR3.3.VCC, CURRENTSENSOR5.A0, CURRENTSENSOR5.IP-, CURRENTSENSOR5.VCC, R10.1, R11.1, R12.1, R13.1, R14.1, R15.1, R7.1, R8.1, R9.1
- net 3.3VACS: no longer CURRENTSENSOR12.IP+, CURRENTSENSOR3.3.IP+, CURRENTSENSOR5.IP+
- net GND: now also C24.2, C25.2, C26.2, C27.2, C28.2, C29.2, C30.-, R22.1, REG-9V.GND1, REG-9V.GND2; no longer CURRENTSENSOR12.A0, CURRENTSENSOR12.GND, CURRENTSENSOR3.3.A0, CURRENTSENSOR3.3.A1, CURRENTSENSOR3.3.GND, CURRENTSENSOR5.A1, CURRENTSENSOR5.GND, R11.2, R12.2, R14.2, R15.2, R8.2, R9.2
- net N$4: now also REG-9V.VOADJUST; no longer REG-12V.VOADJUST
- net VI12V: now also C24.1, C25.1, C26.1, C27.1, REG-9V.VI
Other:
- moved on the sheet: REG-12V

Commit message: edited power supply board sch
Parts:
- removed UVQ: UVQ-24/4.5-D24P-C, murata:UVQ-24/4.5-D24P-C
- added U$3: UWEUWE, murata:UWEUWE
Connections:
- new net UVQ+: U$3.+SENSE, U$3.+VOUT
- new net UVQ-: U$3.-SENSE, U$3.-VOUT
- net UVQV+: no longer UVQ.+VOUT
- net UVQV-: no longer UVQ.-VOUT
Changed lines of the file:
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@@
 <parts>
 <part name="HOTSWAP1" library="linear" deviceset="LTC4231" device=""/>
-<part name="UVQ" library="murata" deviceset="UVQ-24/4.5-D24P-C" device=""/>
 <part name="DIODE-OR-1" library="linear" deviceset="LTC4359" device=""/>
 <part name="JP1" library="samtec" deviceset="MPSC-01-80" device="MPSC-RA-LC"/>
@@
 <part name="C29" library="resistor" deviceset="C-US" device="C0805" value="10 µF"/>
 <part name="C30" library="resistor" deviceset="CPOL-US" device="D" value="100 uF"/>
+<part name="U$3" library="murata" deviceset="UWE" device="UWE"/>
 </parts>
 <sheets>
@@
 <instances>
 <instance part="HOTSWAP1" gate="G$1" x="134.62" y="48.26"/>
-<instance part="UVQ" gate="G$1" x="12.7" y="144.78"/>
 <instance part="DIODE-OR-1" gate="G$1" x="-25.4" y="45.72"/>
 <instance part="JP1" gate="G$1" x="612.14" y="2.54"/>
@@
 <instance part="C29" gate="G$1" x="327.66" y="-96.52" rot="R90"/>
 <instance part="C30" gate="G$1" x="327.66" y="-104.14" rot="R90"/>
+<instance part="U$3" gate="G$1" x="5.08" y="111.76"/>
 </instances>
 <busses>
@@
 <label x="-48.26" y="109.22" size="1.778" layer="95"/>
 </segment>
-<segment>
-<pinref part="UVQ" gate="G$1" pin="+VOUT"/>
-<wire x1="35.56" y1="129.54" x2="63.5" y2="129.54" width="0.1524" layer="91"/>
-<label x="58.42" y="129.54" size="1.778" layer="95"/>
-</segment>
 </net>
 <net name="UVQV-" class="0">
@@
 <wire x1="-50.8" y1="104.14" x2="-45.72" y2="104.14" width="0.1524" layer="91"/>
 <label x="-48.26" y="104.14" size="1.778" layer="95"/>
-</segment>
-<segment>
-<pinref part="UVQ" gate="G$1" pin="-VOUT"/>
-<wire x1="35.56" y1="160.02" x2="63.5" y2="160.02" width="0.1524" layer="91"/>
-<label x="58.42" y="160.02" size="1.778" layer="95"/>
 </segment>
 </net>
@@
 </segment>
 </net>
+<net name="UVQ-" class="0">
+<segment>
+<pinref part="U$3" gate="G$1" pin="-VOUT"/>
+<wire x1="-10.16" y1="104.14" x2="-22.86" y2="104.14" width="0.1524" layer="91"/>
+<pinref part="U$3" gate="G$1" pin="-SENSE"/>
+<wire x1="20.32" y1="119.38" x2="17.78" y2="119.38" width="0.1524" layer="91"/>
+<wire x1="17.78" y1="119.38" x2="17.78" y2="132.08" width="0.1524" layer="91"/>
+<wire x1="17.78" y1="132.08" x2="-22.86" y2="132.08" width="0.1524" layer="91"/>
+<wire x1="-22.86" y1="132.08" x2="-22.86" y2="104.14" width="0.1524" layer="91"/>
+<wire x1="-22.86" y1="104.14" x2="-25.4" y2="104.14" width="0.1524" layer="91"/>
+<junction x="-22.86" y="104.14"/>
+<label x="-30.48" y="104.14" size="1.778" layer="95"/>
+</segment>
+</net>
+<net name="UVQ+" class="0">
+<segment>
+<pinref part="U$3" gate="G$1" pin="+SENSE"/>
+<wire x1="20.32" y1="109.22" x2="27.94" y2="109.22" width="0.1524" layer="91"/>
+<wire x1="27.94" y1="109.22" x2="27.94" y2="96.52" width="0.1524" layer="91"/>
+<wire x1="27.94" y1="96.52" x2="-12.7" y2="96.52" width="0.1524" layer="91"/>
+<pinref part="U$3" gate="G$1" pin="+VOUT"/>
+<wire x1="-12.7" y1="96.52" x2="-20.32" y2="96.52" width="0.1524" layer="91"/>
+<wire x1="20.32" y1="104.14" x2="20.32" y2="99.06" width="0.1524" layer="91"/>
+<wire x1="20.32" y1="99.06" x2="-12.7" y2="99.06" width="0.1524" layer="91"/>
+<wire x1="-12.7" y1="99.06" x2="-12.7" y2="96.52" width="0.1524" layer="91"/>
+<junction x="-12.7" y="96.52"/>
+<label x="-20.32" y="96.52" size="1.778" layer="95"/>
+</segment>
+</net>
