File: Project QUBO/eagleDesigns/powerBoard/testing_board.brd (EAGLE design)
At the start: 160 x 100 mm, 16 parts, among them M1 IRF7458PBF, M2 IRF7458PBF

Commit message: 
Parts:
- R5: value 12K -> 10K
Other:
- board text added: "Designed by Nathaniel Renegar"
- board text added: "R@M 2018"
Changed lines of the file:
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@@
 <wire x1="160" y1="100" x2="0" y2="100" width="0" layer="20"/>
 <wire x1="0" y1="100" x2="0" y2="0" width="0" layer="20"/>
+<text x="36.19" y="60.381" size="0.5" layer="121" font="vector">Designed by Nathaniel Renegar</text>
+<text x="36.195" y="58.801" size="1" layer="121">R@M 2018</text>
 </plain>
 <attributes>
@@
 <element name="R3" library="resistor" package="R0805" value="10K" x="37.211" y="44.958"/>
 <element name="R4" library="resistor" package="R0805" value="10" x="37.211" y="49.911"/>
-<element name="R5" library="resistor" package="R0805" value="12K" x="33.18" y="49.944"/>
+<element name="R5" library="resistor" package="R0805" value="10K" x="33.18" y="49.944"/>
 <element name="R7" library="resistor" package="R0805" value="91K" x="47.752" y="48.006" rot="R270"/>
 <element name="R8" library="resistor" package="R0805" value="5K" x="47.752" y="43.307" rot="R270"/>
