File: Project QUBO/eagleDesigns/powerBoard/testing_board.sch (EAGLE design)
At the start: 16 parts, among them M1 IRF7458PBF, M2 IRF7458PBF

Commit message: 
Parts:
- R5: value 12K -> 10K
Changed lines of the file:
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@@
 <part name="GND1" library="supply1" deviceset="GND" device=""/>
 <part name="R4" library="resistor" deviceset="R-US_" device="R0805" value="10"/>
-<part name="R5" library="resistor" deviceset="R-US_" device="R0805" value="12K"/>
+<part name="R5" library="resistor" deviceset="R-US_" device="R0805" value="10K"/>
 <part name="C3" library="resistor" deviceset="C-EU" device="C0805" value="6.8nF"/>
 <part name="C4" library="resistor" deviceset="C-EU" device="C0805" value="22uF"/>
