File: Project QUBO/eagleDesigns/backplane/version2/backplane_v3.sch (EAGLE design)
At the start: 88 parts

Commit message: 
Parts:
- added 2PIN_1: CPU_USB_HUB, molex:KK254_VERT_2PIN22-29-2021
- added 2PIN_2: CPU_USB_AHRS, molex:KK254_VERT_2PIN22-29-2021
- added 2PIN_3: CPU_USB_IMU, molex:KK254_VERT_2PIN22-29-2021
- added 2PIN_4: CPU_USB_To-DVL, molex:KK254_VERT_2PIN22-29-2021
- added 2PIN_5: CPU_USB_From-DVL, molex:KK254_VERT_2PIN22-29-2021
- added 2PIN_6: CPU_I2C_1, molex:KK254_VERT_2PIN22-29-2021
- added 4PIN_1: CPU_RS232_MCU, molex:KK254_VERT_4PIN22-29-2041
- added 4PIN_2: CPU_RS232_Flex, molex:KK254_VERT_4PIN22-29-2041
- added 4PIN_3: CPU_PWR1, molex:KK254_VERT_4PIN22-29-2041
- added 4PIN_4: CPU_PWR2, molex:KK254_VERT_4PIN22-29-2041
- added 4PIN_5: CPU_GND1, molex:KK254_VERT_4PIN22-29-2041
- added 4PIN_6: CPU_GND2, molex:KK254_VERT_4PIN22-29-2041
- added U$15: SPI_LEDS, molex:KK254_6PIN
- added U$16: CPU_SPI, molex:KK254_6PIN
- SPI_LEDS: value KK254_6PIN -> (none)
Connections:
- new net N$64: U$15.P$6
- new net N$65: U$15.P$5
- new net N$66: U$15.P$4
- new net N$68: U$15.P$3
- new net N$69: U$15.P$2
- new net N$70: U$15.P$1
- net GND: now also 4PIN_5.P$1, 4PIN_5.P$2, 4PIN_5.P$3, 4PIN_5.P$4, 4PIN_6.P$1, 4PIN_6.P$2, 4PIN_6.P$3, 4PIN_6.P$4
- net V_BATT: now also 4PIN_3.P$1, 4PIN_3.P$2, 4PIN_3.P$3, 4PIN_3.P$4, 4PIN_4.P$1, 4PIN_4.P$2, 4PIN_4.P$3, 4PIN_4.P$4
Changed lines of the file:
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@@
 <part name="U$13" library="NXP" deviceset="PRTR5V0U2X" device=""/>
 <part name="U$14" library="NXP" deviceset="PRTR5V0U2X" device=""/>
+<part name="2PIN_1" library="molex" deviceset="KK254_VERT_2PIN" device="22-29-2021" value="CPU_USB_HUB"/>
+<part name="2PIN_2" library="molex" deviceset="KK254_VERT_2PIN" device="22-29-2021" value="CPU_USB_AHRS"/>
+<part name="2PIN_3" library="molex" deviceset="KK254_VERT_2PIN" device="22-29-2021" value="CPU_USB_IMU"/>
+<part name="2PIN_4" library="molex" deviceset="KK254_VERT_2PIN" device="22-29-2021" value="CPU_USB_To-DVL"/>
+<part name="2PIN_5" library="molex" deviceset="KK254_VERT_2PIN" device="22-29-2021" value="CPU_USB_From-DVL"/>
+<part name="4PIN_1" library="molex" deviceset="KK254_VERT_4PIN" device="22-29-2041" value="CPU_RS232_MCU"/>
+<part name="4PIN_2" library="molex" deviceset="KK254_VERT_4PIN" device="22-29-2041" value="CPU_RS232_Flex"/>
+<part name="2PIN_6" library="molex" deviceset="KK254_VERT_2PIN" device="22-29-2021" value="CPU_I2C_1"/>
+<part name="U$15" library="molex" deviceset="KK254_6PIN" device="" value="SPI_LEDS"/>
+<part name="U$16" library="molex" deviceset="KK254_6PIN" device="" value="CPU_SPI"/>
+<part name="4PIN_3" library="molex" deviceset="KK254_VERT_4PIN" device="22-29-2041" value="CPU_PWR1"/>
+<part name="4PIN_4" library="molex" deviceset="KK254_VERT_4PIN" device="22-29-2041" value="CPU_PWR2"/>
+<part name="4PIN_5" library="molex" deviceset="KK254_VERT_4PIN" device="22-29-2041" value="CPU_GND1"/>
+<part name="4PIN_6" library="molex" deviceset="KK254_VERT_4PIN" device="22-29-2041" value="CPU_GND2"/>
 </parts>
 <sheets>
@@
 <instance part="U$13" gate="G$1" x="-162.56" y="-330.2"/>
 <instance part="U$14" gate="G$1" x="-231.14" y="-363.22"/>
+<instance part="2PIN_1" gate="U1" x="-787.4" y="25.4"/>
+<instance part="2PIN_2" gate="U1" x="-787.4" y="-2.54"/>
+<instance part="2PIN_3" gate="U1" x="-787.4" y="-30.48"/>
+<instance part="2PIN_4" gate="U1" x="-787.4" y="-58.42"/>
+<instance part="2PIN_5" gate="U1" x="-787.4" y="-86.36"/>
+<instance part="4PIN_1" gate="U1" x="-787.4" y="-116.84"/>
+<instance part="4PIN_2" gate="U1" x="-787.4" y="-147.32"/>
+<instance part="2PIN_6" gate="U1" x="-787.4" y="-177.8"/>
+<instance part="U$15" gate="G$1" x="-787.4" y="-213.36"/>
+<instance part="U$16" gate="G$1" x="-858.52" y="-213.36"/>
+<instance part="4PIN_3" gate="U1" x="-787.4" y="-264.16"/>
+<instance part="4PIN_4" gate="U1" x="-858.52" y="-266.7"/>
+<instance part="4PIN_5" gate="U1" x="-787.4" y="-307.34"/>
+<instance part="4PIN_6" gate="U1" x="-858.52" y="-307.34"/>
 </instances>
 <busses>
@@
 <label x="-248.92" y="-358.14" size="1.778" layer="95"/>
 </segment>
+<segment>
+<pinref part="4PIN_5" gate="U1" pin="P$4"/>
+<pinref part="4PIN_5" gate="U1" pin="P$1"/>
+<wire x1="-795.02" y1="-302.26" x2="-795.02" y2="-304.8" width="0.1524" layer="91"/>
+<wire x1="-795.02" y1="-304.8" x2="-795.02" y2="-309.88" width="0.1524" layer="91"/>
+<wire x1="-795.02" y1="-309.88" x2="-795.02" y2="-312.42" width="0.1524" layer="91"/>
+<wire x1="-795.02" y1="-312.42" x2="-802.64" y2="-312.42" width="0.1524" layer="91"/>
+<junction x="-795.02" y="-312.42"/>
+<pinref part="4PIN_5" gate="U1" pin="P$2"/>
+<junction x="-795.02" y="-309.88"/>
+<pinref part="4PIN_5" gate="U1" pin="P$3"/>
+<junction x="-795.02" y="-304.8"/>
+<label x="-802.64" y="-312.42" size="1.778" layer="95"/>
+</segment>
+<segment>
+<pinref part="4PIN_6" gate="U1" pin="P$4"/>
+<pinref part="4PIN_6" gate="U1" pin="P$1"/>
+<wire x1="-866.14" y1="-302.26" x2="-866.14" y2="-304.8" width="0.1524" layer="91"/>
+<wire x1="-866.14" y1="-304.8" x2="-866.14" y2="-309.88" width="0.1524" layer="91"/>
+<wire x1="-866.14" y1="-309.88" x2="-866.14" y2="-312.42" width="0.1524" layer="91"/>
+<wire x1="-866.14" y1="-312.42" x2="-873.76" y2="-312.42" width="0.1524" layer="91"/>
+<junction x="-866.14" y="-312.42"/>
+<label x="-873.76" y="-312.42" size="1.778" layer="95"/>
+<pinref part="4PIN_6" gate="U1" pin="P$2"/>
+<junction x="-866.14" y="-309.88"/>
+<pinref part="4PIN_6" gate="U1" pin="P$3"/>
+<junction x="-866.14" y="-304.8"/>
+</segment>
 </net>
 <net name="3V3" class="0">
@@
 <label x="177.8" y="-127" size="1.778" layer="95"/>
 </segment>
+<segment>
+<pinref part="4PIN_4" gate="U1" pin="P$4"/>
+<pinref part="4PIN_4" gate="U1" pin="P$1"/>
+<wire x1="-866.14" y1="-261.62" x2="-866.14" y2="-264.16" width="0.1524" layer="91"/>
+<wire x1="-866.14" y1="-264.16" x2="-866.14" y2="-269.24" width="0.1524" layer="91"/>
+<wire x1="-866.14" y1="-269.24" x2="-866.14" y2="-271.78" width="0.1524" layer="91"/>
+<wire x1="-866.14" y1="-271.78" x2="-873.76" y2="-271.78" width="0.1524" layer="91"/>
+<junction x="-866.14" y="-271.78"/>
+<label x="-876.3" y="-271.78" size="1.778" layer="95"/>
+<pinref part="4PIN_4" gate="U1" pin="P$2"/>
+<junction x="-866.14" y="-269.24"/>
+<pinref part="4PIN_4" gate="U1" pin="P$3"/>
+<junction x="-866.14" y="-264.16"/>
+</segment>
+<segment>
+<pinref part="4PIN_3" gate="U1" pin="P$4"/>
+<pinref part="4PIN_3" gate="U1" pin="P$1"/>
+<wire x1="-795.02" y1="-259.08" x2="-795.02" y2="-261.62" width="0.1524" layer="91"/>
+<pinref part="4PIN_3" gate="U1" pin="P$2"/>
+<junction x="-795.02" y="-266.7"/>
+<wire x1="-795.02" y1="-261.62" x2="-795.02" y2="-266.7" width="0.1524" layer="91"/>
+<wire x1="-795.02" y1="-266.7" x2="-795.02" y2="-269.24" width="0.1524" layer="91"/>
+<pinref part="4PIN_3" gate="U1" pin="P$3"/>
+<junction x="-795.02" y="-261.62"/>
+<wire x1="-795.02" y1="-269.24" x2="-805.18" y2="-269.24" width="0.1524" layer="91"/>
+<junction x="-795.02" y="-269.24"/>
+<label x="-805.18" y="-269.24" size="1.778" layer="95"/>
+</segment>
 </net>
 <net name="CTS_4" class="0">
@@
 </segment>
 </net>
+<net name="N$64" class="0">
+<segment>
+<pinref part="U$15" gate="G$1" pin="P$6"/>
+<wire x1="-795.02" y1="-205.74" x2="-812.8" y2="-205.74" width="0.1524" layer="91"/>
+</segment>
+</net>
+<net name="N$65" class="0">
+<segment>
+<pinref part="U$15" gate="G$1" pin="P$5"/>
+<wire x1="-795.02" y1="-208.28" x2="-812.8" y2="-208.28" width="0.1524" layer="91"/>
+</segment>
+</net>
+<net name="N$66" class="0">
+<segment>
+<pinref part="U$15" gate="G$1" pin="P$4"/>
+<wire x1="-795.02" y1="-210.82" x2="-812.8" y2="-210.82" width="0.1524" layer="91"/>
+</segment>
+</net>
+<net name="N$68" class="0">
+<segment>
+<pinref part="U$15" gate="G$1" pin="P$3"/>
+<wire x1="-795.02" y1="-215.9" x2="-812.8" y2="-215.9" width="0.1524" layer="91"/>
+</segment>
+</net>
+<net name="N$69" class="0">
+<segment>
+<pinref part="U$15" gate="G$1" pin="P$2"/>
+<wire x1="-795.02" y1="-218.44" x2="-812.8" y2="-218.44" width="0.1524" layer="91"/>
+</segment>
+</net>
+<net name="N$70" class="0">
+<segment>
+<pinref part="U$15" gate="G$1" pin="P$1"/>
+<wire x1="-795.02" y1="-220.98" x2="-812.8" y2="-220.98" width="0.1524" layer="91"/>
+</segment>
+</net>

Commit message: 
Parts:
- removed 2PIN_4: CPU_USB_To-DVL, molex:KK254_VERT_2PIN22-29-2021
- removed SPI_LEDS: (no value), molex:KK254_6PIN
- removed U$16: CPU_SPI, molex:KK254_6PIN
- added 2PIN_7: CPU_CAN, molex:KK254_VERT_2PIN22-29-2021
- added 4PIN_7: CPU_SPI, molex:KK254_VERT_4PIN22-29-2041
- 2PIN_5: value CPU_USB_From-DVL -> CPU_USB_DVL
Connections:
- removed net CE_1: JP1.P$53, JP2.P$53, JP3.P$53, JP4.P$53
- removed net CE_DEBUG-LEDS: JP1.P$52, JP2.P$52, JP3.P$52, JP4.P$52, SPI_LEDS.P$1
- removed net FLEX_USB_1+\: JP1.P$17, JP2.P$17, JP3.P$17, JP4.P$17
- removed net FLEX_USB_1-: JP1.P$16, JP2.P$16, JP3.P$16, JP4.P$16
- removed net FLEX_USB_2+: JP1.P$14, JP2.P$14, JP3.P$14, JP4.P$14
- removed net FLEX_USB_2-: JP1.P$13, JP2.P$13, JP3.P$13, JP4.P$13
- removed net IMUT_USB-: IMU_FTDI.USBDM
- removed net N$64: U$15.P$6
- removed net N$65: U$15.P$5
- removed net N$66: U$15.P$4
- removed net N$68: U$15.P$3
- removed net N$69: U$15.P$2
- removed net N$70: U$15.P$1
- new net AHRS_USB+: 2PIN_2.P$1
- new net AHRS_USB-: 2PIN_2.P$2
- new net CE_CPU: 4PIN_7.P$2, JP1.P$53, JP2.P$53, JP3.P$53, JP4.P$53
- new net CE_LEDS: JP1.P$52, JP2.P$52, JP3.P$52, JP4.P$52, U$15.P$3
- new net HUB_USB+: 2PIN_1.P$1
- new net HUB_USB-: 2PIN_1.P$2
- new net IMU_USB-: 2PIN_3.P$2, IMU_FTDI.USBDM
- new net NC: JP1.P$13, JP1.P$14, JP1.P$16, JP1.P$17, JP2.P$13, JP2.P$14, JP2.P$16, JP2.P$17, JP3.P$13, JP3.P$14, JP3.P$16, JP3.P$17, JP4.P$13, JP4.P$14, JP4.P$16, JP4.P$17
- net 12V: now also U$15.P$2
- net 5V: no longer SPI_LEDS.P$6
- net CANH: now also 2PIN_7.P$2
- net CANL: now also 2PIN_7.P$1
- net CTS_2: now also 4PIN_1.P$1
- net CTS_3: now also 4PIN_2.P$1
- net DVL_USB+: now also 2PIN_5.P$1
- net DVL_USB-: now also 2PIN_5.P$2
- net GND: now also U$15.P$1; no longer SPI_LEDS.P$5
- net IMU_USB+: now also 2PIN_3.P$1
- net MISO: now also 4PIN_7.P$3, U$15.P$5; no longer SPI_LEDS.P$2
- net MOSI: now also 4PIN_7.P$4, U$15.P$6; no longer SPI_LEDS.P$3
- net RTS_2: now also 4PIN_1.P$2
- net RTS_3: now also 4PIN_2.P$2
- net RX_2: now also 4PIN_1.P$4
- net RX_3: now also 4PIN_2.P$4
- net SCL_1: now also 2PIN_6.P$1
- net SDA_1: now also 2PIN_6.P$2
- net SPI_CLK: now also 4PIN_7.P$1, U$15.P$4; no longer SPI_LEDS.P$4
- net TX_2: now also 4PIN_1.P$3
- net TX_3: now also 4PIN_2.P$3
Other:
- moved on the sheet: 2PIN_1, 2PIN_2, 2PIN_3, 2PIN_5, 4PIN_3, 4PIN_4, 4PIN_5, 4PIN_6, U$15

Commit message: 
Parts:
- removed C2, C3: (no value), resistor:C-USC0805
- removed CPU_USB_CPU: (no value), molex:KK254_VERT_2PIN22-29-2021
- removed R2: 27, resistor:R-US_R0805
- removed U$14: PRTR5V0U2X, NXP:PRTR5V0U2X
- added G1: (no value), texas:TPS2044BBD-SOIC
- added IC1: MC78M08ABDTG, linear:MC78M08ABDTG
- added U1: TUSB2077ALQFP, texas:TUSB2077ALQFP
- R1: value 27 -> 120
- U$1: value USB2517-JZX -> 24MHz; device microchip:USB2517-JZX -> microchip:DCS6XXX
- U$10: value PRTR5V0U2X -> (none); device NXP:PRTR5V0U2X -> hirose:HR30-6R-6PD
- U$11, U$12: value PRTR5V0U2X -> 1U_tant; device NXP:PRTR5V0U2X -> avx:F93-XX-XXX-X-A
- U$13: value PRTR5V0U2X -> MEMSENSE_NIMU; device NXP:PRTR5V0U2X -> nonelectrical_mounting:MEMSENSE_NIMU
Connections:
- net DVL_HUSB+ renamed DVL_HUSB_P
- net DVL_HUSB- renamed DVL_HUSB_M
- net DVL_SUSB+ renamed DVL_SUSB_P
- net DVL_SUSB- renamed DVL_SUSB_M
- net IMU_RXD renamed IMU_RX
- net USB_1+ renamed USB_1_P
- net USB_1- renamed USB_1_M
- net USB_2+ renamed USB_2_P
- net USB_2- renamed USB_2_M
- net USB_3+ renamed USB_3_P
- net USB_3- renamed USB_3_M
- net USB_4+ renamed USB_4_P
- net USB_4- renamed USB_4_M
- removed net AHRS_USB+: 2PIN_2.P$1
- removed net AHRS_USB-: 2PIN_2.P$2
- removed net CPU_USB_CPU_D+: C3.1, R1.2
- removed net CPU_USB_CPU_D-: C2.1, R2.2
- removed net DVL_USB+: 2PIN_5.P$1, DVL_USB_HUB.USBDP_UP
- removed net DVL_USB-: 2PIN_5.P$2, DVL_USB_HUB.USBDM_UP
- removed net HUB_USB+: 2PIN_1.P$1
- removed net HUB_USB-: 2PIN_1.P$2
- removed net IMU_RX-A: IMU_TTL-TO-RS422.R1-IN/(A)
- removed net IMU_RX-B: IMU_TTL-TO-RS422.R1-IN(B)
- removed net IMU_USB+: 2PIN_3.P$1, IMU_FTDI.USBDP
- removed net IMU_USB-: 2PIN_3.P$2, IMU_FTDI.USBDM
- removed net N$1: U$3.I/O_1
- removed net N$10: U$5.I/O_1
- removed net N$11: U$5.I/O_2
- removed net N$12: U$6.I/O_1
- removed net N$13: U$6.I/O_2
- removed net N$14: U$7.I/O_1
- removed net N$15: U$7.I/O_2
- removed net N$18: U$9.I/O_1
- removed net N$19: CPU_USB_CPU.P$1, R2.1
- removed net N$2: U$2.I/O_1
- removed net N$20: U$9.I/O_2
- removed net N$21: U$10.I/O_1
- removed net N$47: U$10.I/O_2
- removed net N$48: U$11.I/O_1
- removed net N$5: CPU_USB_CPU.P$2, R1.1
- removed net N$50: U$11.I/O_2
- removed net N$51: U$12.I/O_1
- removed net N$53: DVL_USB_HUB.XTALIN/CLO\KIN
- removed net N$58: U$12.I/O_2
- removed net N$6: U$3.I/O_2
- removed net N$60: U$13.I/O_1
- removed net N$61: U$13.I/O_2
- removed net N$62: U$14.I/O_1
- removed net N$63: U$14.I/O_2
- removed net N$7: U$2.I/O_2
- removed net USB_EXT+: 5.7.P$2
- removed net USB_EXT-: 5.7.P$1
- new net 8V: IC1.VO, U$10.2, U$12.+
- new net AHRS_USB_M: 2PIN_2.P$2, U$6.I/O_2
- new net AHRS_USB_P: 2PIN_2.P$1, U$6.I/O_1
- new net DVL_USB_HUB_XTAL: DVL_USB_HUB.XTALIN/CLO\KIN, U$1.OUT
- new net DVL_USB_M: 2PIN_5.P$2, DVL_USB_HUB.USBDM_UP, U$7.I/O_2
- new net DVL_USB_P: 2PIN_5.P$1, DVL_USB_HUB.USBDP_UP, U$7.I/O_1
- new net EXT_USB_M: 5.7.P$1, U$5.I/O_2
- new net EXT_USB_P: 5.7.P$2, U$5.I/O_1
- new net HUB_USB_M: 2PIN_1.P$2, U$2.I/O_2
- new net HUB_USB_P: 2PIN_1.P$1, U$2.I/O_1
- new net IMU_RXD_M: IMU_TTL-TO-RS422.R1-IN(B), R1.1, U$10.4, U$9.I/O_2
- new net IMU_RXD_P: IMU_TTL-TO-RS422.R1-IN/(A), R1.2, U$10.3, U$9.I/O_1
- new net IMU_USB_M: 2PIN_3.P$2, IMU_FTDI.USBDM, U$3.I/O_2
- new net IMU_USB_P: 2PIN_3.P$1, IMU_FTDI.USBDP, U$3.I/O_1
- net 12V: now also IC1.VI, U$11.+
- net 3V3: now also U$1.EN, U$1.VDD; no longer U$10.VCC, U$11.VCC, U$12.VCC, U$13.VCC, U$14.VCC
- net GND: now also IC1.GND, U$1.GND, U$10.5, U$11.-, U$12.-; no longer C2.2, C3.2, U$10.GND, U$11.GND, U$12.GND, U$13.GND, U$14.GND
Other:
- note added: "IMU Connection"
- moved on the sheet: R1, U$15, U$2, U$3, U$5, U$6, U$7, U$9
