File: Project QUBO/eagleDesigns/backplane/version2/backplane_v4.sch (EAGLE design)
At the start: 302 parts, among them U1 TUSB2077ALQFP

Commit message: 
Connections:
- net RTS_0 renamed RX_SF
- net SCL_0_UNBUF renamed BATT_SCL_UNBUF
- net SDA_0_UNBUF renamed BATT_SDA_UNBUF
- removed net CTS_0: JP1.P$47, JP2.P$47, JP3.P$47, JP4.P$47
- removed net CTS_1: JP1.P$31, JP2.P$31, JP3.P$31, JP4.P$31
- removed net CTS_2: 4PIN_1.P$1, JP1.P$71, JP2.P$71, JP3.P$71, JP4.P$71
- removed net CTS_3: 4PIN_2.P$1, JP1.P$75, JP2.P$75, JP3.P$75, JP4.P$75
- removed net CTS_4: JP1.P$79, JP2.P$79, JP3.P$79, JP4.P$79
- removed net CTS_5: 5.2.P$3, JP1.P$67, JP2.P$67, JP3.P$67, JP4.P$67, U$55.I/O_2
- removed net GND\: DVL_USB_HUB.GND, JP1.P$40, JP2.P$40, JP3.P$40, JP4.P$40
- removed net GPIO_0: JP1.P$35, JP2.P$35, JP3.P$35, JP4.P$35
- removed net GPIO_1: JP1.P$38, JP2.P$38, JP3.P$38, JP4.P$38
- removed net GPIO_3: JP1.P$57, JP2.P$57, JP3.P$57, JP4.P$57
- removed net GPIO_4: JP1.P$58, JP2.P$58, JP3.P$58, JP4.P$58
- removed net NC: JP1.P$13, JP1.P$14, JP1.P$16, JP1.P$17, JP2.P$13, JP2.P$14, JP2.P$16, JP2.P$17, JP3.P$13, JP3.P$14, JP3.P$16, JP3.P$17, JP4.P$13, JP4.P$14, JP4.P$16, JP4.P$17
- removed net RTS_1: JP1.P$32, JP2.P$32, JP3.P$32, JP4.P$32
- removed net RTS_2: 4PIN_1.P$2, JP1.P$72, JP2.P$72, JP3.P$72, JP4.P$72
- removed net RTS_3: 4PIN_2.P$2, JP1.P$76, JP2.P$76, JP3.P$76, JP4.P$76
- removed net RTS_4: JP1.P$80, JP2.P$80, JP3.P$80, JP4.P$80
- removed net RTS_5: 5.2.P$4, JP1.P$68, JP2.P$68, JP3.P$68, JP4.P$68, U$55.I/O_1
- removed net RX_0: JP1.P$45, JP2.P$45, JP3.P$45, JP4.P$45
- removed net RX_1: JP1.P$29, JP2.P$29, JP3.P$29, JP4.P$29
- removed net RX_2: 4PIN_1.P$4, JP1.P$69, JP2.P$69, JP3.P$69, JP4.P$69, U$4.I/O_2
- removed net RX_3: 4PIN_2.P$4, JP1.P$73, JP2.P$73, JP3.P$73, JP4.P$73, U$8.I/O_1
- removed net RX_4: JP1.P$77, JP2.P$77, JP3.P$77, JP4.P$77
- removed net RX_5: 5.2.P$1, JP1.P$65, JP2.P$65, JP3.P$65, JP4.P$65, U$54.I/O_1
- removed net SCL_0: JP1.P$28, JP2.P$28, JP3.P$28, JP4.P$28, U$38.LX
- removed net SCL_1: 2PIN_6.P$1, JP1.P$10, JP2.P$10, JP3.P$10, JP4.P$10, U$18.I/O_1, U$50.LX
- removed net SCL_2: 5.4.P$5, JP1.P$60, JP2.P$60, JP3.P$60, JP4.P$60, U$63.I/O_1
- removed net SCL_3: 5.3.P$2, JP1.P$6, JP2.P$6, JP3.P$6, JP4.P$6, U$52.I/O_1
- removed net SDA_0: JP1.P$27, JP2.P$27, JP3.P$27, JP4.P$27, U$38.LY
- removed net SDA_1: 2PIN_6.P$2, JP1.P$9, JP2.P$9, JP3.P$9, JP4.P$9, U$18.I/O_2, U$50.LY
- removed net SDA_2: 5.5.P$5, JP1.P$59, JP2.P$59, JP3.P$59, JP4.P$59, U$63.I/O_2
- removed net SDA_3: 5.3.P$1, JP1.P$5, JP2.P$5, JP3.P$5, JP4.P$5, U$52.I/O_2
- removed net TX_0: JP1.P$46, JP2.P$46, JP3.P$46, JP4.P$46
- removed net TX_1: JP1.P$30, JP2.P$30, JP3.P$30, JP4.P$30
- removed net TX_2: 4PIN_1.P$3, JP1.P$70, JP2.P$70, JP3.P$70, JP4.P$70, U$4.I/O_1
- removed net TX_3: 4PIN_2.P$3, JP1.P$74, JP2.P$74, JP3.P$74, JP4.P$74, U$8.I/O_2
- removed net TX_4: JP1.P$78, JP2.P$78, JP3.P$78, JP4.P$78
- removed net TX_5: 5.2.P$2, JP1.P$66, JP2.P$66, JP3.P$66, JP4.P$66, U$54.I/O_2
- removed net USB_1_M: JP1.P$19, R2.1, R22.1, U$29.I/O_2
- removed net USB_2_M: JP2.P$19, R24.1, R37.1, U$30.I/O_2
- removed net USB_3_M: JP3.P$19, R27.2, R40.1, U$31.I/O_2
- removed net USB_4_M: JP4.P$19, R28.2, R41.1, U$32.I/O_2
- new net ACT_SCL: 5.4.P$5, JP1.P$24, JP2.P$24, JP3.P$24, JP4.P$24, U$63.I/O_1
- new net ACT_SDA: 5.5.P$5, JP1.P$23, JP2.P$23, JP3.P$23, JP4.P$23, U$63.I/O_2
- new net BATT_SCL: JP1.P$44, JP2.P$44, JP3.P$44, JP4.P$44, U$38.LX
- new net BATT_SDA: JP1.P$43, JP2.P$43, JP3.P$43, JP4.P$43, U$38.LY
- new net CTS_CF: 4PIN_2.P$1, JP1.P$13, JP2.P$13, JP3.P$13, JP4.P$13
- new net CTS_MC: 4PIN_1.P$1, JP1.P$29, JP2.P$29, JP3.P$29, JP4.P$29
- new net CTS_MD: 5.2.P$3, JP1.P$68, JP2.P$68, JP3.P$68, JP4.P$68, U$55.I/O_2
- new net CTS_MF: JP1.P$5, JP2.P$5, JP3.P$5, JP4.P$5
- new net CTS_PF: JP1.P$9, JP2.P$9, JP3.P$9, JP4.P$9
- new net CTS_SF: JP1.P$50, JP2.P$50, JP3.P$50, JP4.P$50
- new net EXT_SCL: 5.3.P$2, JP1.P$34, JP2.P$34, JP3.P$34, JP4.P$34, U$52.I/O_1
- new net EXT_SDA: 5.3.P$1, JP1.P$33, JP2.P$33, JP3.P$33, JP4.P$33, U$52.I/O_2
- new net GPIO_22: JP1.P$22, JP2.P$22, JP3.P$22, JP4.P$22
- new net GPIO_63: JP1.P$63, JP2.P$63, JP3.P$63, JP4.P$63
- new net INT_SCL: 2PIN_6.P$1, JP1.P$65, JP2.P$65, JP3.P$65, JP4.P$65, U$18.I/O_1, U$50.LX
- new net INT_SDA: 2PIN_6.P$2, JP1.P$64, JP2.P$64, JP3.P$64, JP4.P$64, U$18.I/O_2, U$50.LY
- new net RTS_CF: 4PIN_2.P$2, JP1.P$14, JP2.P$14, JP3.P$14, JP4.P$14
- new net RTS_MC: 4PIN_1.P$2, JP1.P$30, JP2.P$30, JP3.P$30, JP4.P$30
- new net RTS_MD: 5.2.P$4, JP1.P$69, JP2.P$69, JP3.P$69, JP4.P$69, U$55.I/O_1
- new net RTS_MF: JP1.P$6, JP2.P$6, JP3.P$6, JP4.P$6
- new net RTS_PF: JP1.P$10, JP2.P$10, JP3.P$10, JP4.P$10
- new net RTS_SF: JP1.P$51, JP2.P$51, JP3.P$51, JP4.P$51
- new net RX_CF: 4PIN_2.P$4, JP1.P$11, JP2.P$11, JP3.P$11, JP4.P$11, U$8.I/O_1
- new net RX_MC: 4PIN_1.P$4, JP1.P$27, JP2.P$27, JP3.P$27, JP4.P$27, U$4.I/O_2
- new net RX_MD: 5.2.P$1, JP1.P$66, JP2.P$66, JP3.P$66, JP4.P$66, U$54.I/O_1
- new net RX_MF: JP1.P$3, JP2.P$3, JP3.P$3, JP4.P$3
- new net RX_PF: JP1.P$7, JP2.P$7, JP3.P$7, JP4.P$7
- new net TX_CF: 4PIN_2.P$3, JP1.P$12, JP2.P$12, JP3.P$12, JP4.P$12, U$8.I/O_2
- new net TX_MC: 4PIN_1.P$3, JP1.P$28, JP2.P$28, JP3.P$28, JP4.P$28, U$4.I/O_1
- new net TX_MD: 5.2.P$2, JP1.P$67, JP2.P$67, JP3.P$67, JP4.P$67, U$54.I/O_2
- new net TX_MF: JP1.P$4, JP2.P$4, JP3.P$4, JP4.P$4
- new net TX_PF: JP1.P$8, JP2.P$8, JP3.P$8, JP4.P$8
- new net TX_SF: JP1.P$49, JP2.P$49, JP3.P$49, JP4.P$49
- new net USB_1_N: JP1.P$61, R2.1, R22.1, U$29.I/O_2
- new net USB_2_N: JP2.P$61, R24.1, R37.1, U$30.I/O_2
- new net USB_3_N: JP3.P$61, R27.2, R40.1, U$31.I/O_2
- new net USB_4_N: JP4.P$61, R28.2, R41.1, U$32.I/O_2
- net 12V: now also JP1.P$16, JP1.P$36, JP1.P$56, JP1.P$76, JP2.P$16, JP2.P$36, JP2.P$56, JP2.P$76, JP3.P$16, JP3.P$36, JP3.P$56, JP3.P$76, JP4.P$16, JP4.P$36, JP4.P$56, JP4.P$76; no longer JP1.P$1, JP1.P$21, JP1.P$41, JP1.P$61, JP2.P$1, JP2.P$21, JP2.P$41, JP2.P$61, JP3.P$1, JP3.P$21, JP3.P$41, JP3.P$61, JP4.P$1, JP4.P$21, JP4.P$41, JP4.P$61
- net 3V3: now also JP1.P$18, JP1.P$38, JP1.P$58, JP1.P$78, JP2.P$18, JP2.P$38, JP2.P$58, JP2.P$78, JP3.P$18, JP3.P$38, JP3.P$58, JP3.P$78, JP4.P$18, JP4.P$38, JP4.P$58, JP4.P$78; no longer JP1.P$23, JP1.P$3, JP1.P$43, JP1.P$63, JP2.P$23, JP2.P$3, JP2.P$43, JP2.P$63, JP3.P$23, JP3.P$3, JP3.P$43, JP3.P$63, JP4.P$23, JP4.P$3, JP4.P$43, JP4.P$63
- net 5V: now also JP1.P$17, JP1.P$37, JP1.P$57, JP1.P$77, JP2.P$17, JP2.P$37, JP2.P$57, JP2.P$77, JP3.P$17, JP3.P$37, JP3.P$57, JP3.P$77, JP4.P$17, JP4.P$37, JP4.P$57, JP4.P$77; no longer JP1.P$2, JP1.P$22, JP1.P$42, JP1.P$62, JP2.P$2, JP2.P$22, JP2.P$42, JP2.P$62, JP3.P$2, JP3.P$22, JP3.P$42, JP3.P$62, JP4.P$2, JP4.P$22, JP4.P$42, JP4.P$62
- net CANH: now also JP1.P$45, JP2.P$45, JP3.P$45, JP4.P$45; no longer JP1.P$25, JP2.P$25, JP3.P$25, JP4.P$25
- net CANL: now also JP1.P$46, JP2.P$46, JP3.P$46, JP4.P$46; no longer JP1.P$26, JP2.P$26, JP3.P$26, JP4.P$26
- net CE_2: now also JP1.P$52, JP2.P$52, JP3.P$52, JP4.P$52; no longer JP1.P$54, JP2.P$54, JP3.P$54, JP4.P$54
- net CE_3: now also JP1.P$53, JP2.P$53, JP3.P$53, JP4.P$53; no longer JP1.P$55, JP2.P$55, JP3.P$55, JP4.P$55
- net CE_4: now also JP1.P$54, JP2.P$54, JP3.P$54, JP4.P$54; no longer JP1.P$56, JP2.P$56, JP3.P$56, JP4.P$56
- net CE_CPU: now also JP1.P$74, JP2.P$74, JP3.P$74, JP4.P$74; no longer JP1.P$53, JP2.P$53, JP3.P$53, JP4.P$53
- net CE_LEDS: now also JP1.P$73, JP2.P$73, JP3.P$73, JP4.P$73; no longer JP1.P$52, JP2.P$52, JP3.P$52, JP4.P$52
- net GND: now also DVL_USB_HUB.GND, JP1.P$1, JP1.P$19, JP1.P$20, JP1.P$21, JP1.P$25, JP1.P$32, JP1.P$35, JP1.P$40, JP1.P$42, JP1.P$47, JP1.P$55, JP1.P$59, JP1.P$60, JP1.P$62, JP1.P$75, JP1.P$79, JP1.P$80, JP1.POWER1, JP2.P$1, JP2.P$19, JP2.P$20, JP2.P$21, JP2.P$25, JP2.P$32, JP2.P$35, JP2.P$40, JP2.P$42, JP2.P$47, JP2.P$55, JP2.P$59, JP2.P$60, JP2.P$62, JP2.P$75, JP2.P$79, JP2.P$80, JP2.POWER1, JP3.P$1, JP3.P$19, JP3.P$20, JP3.P$21, JP3.P$25, JP3.P$32, JP3.P$35, JP3.P$40, JP3.P$42, JP3.P$47, JP3.P$55, JP3.P$59, JP3.P$60, JP3.P$62, JP3.P$75, JP3.P$79, JP3.P$80, JP3.POWER1, JP4.P$1, JP4.P$19, JP4.P$20, JP4.P$21, JP4.P$25, JP4.P$32, JP4.P$35, JP4.P$40, JP4.P$42, JP4.P$47, JP4.P$55, JP4.P$59, JP4.P$60, JP4.P$62, JP4.P$75, JP4.P$79, JP4.P$80, JP4.POWER1; no longer JP1.P$12, JP1.P$18, JP1.P$24, JP1.P$33, JP1.P$34, JP1.P$36, JP1.P$37, JP1.P$4, JP1.P$44, JP1.P$64, JP1.POWER2, JP2.P$12, JP2.P$18, JP2.P$24, JP2.P$33, JP2.P$34, JP2.P$36, JP2.P$37, JP2.P$4, JP2.P$44, JP2.P$64, JP2.POWER2, JP3.P$12, JP3.P$18, JP3.P$24, JP3.P$33, JP3.P$34, JP3.P$36, JP3.P$37, JP3.P$4, JP3.P$44, JP3.P$64, JP3.POWER2, JP4.P$12, JP4.P$18, JP4.P$24, JP4.P$33, JP4.P$34, JP4.P$36, JP4.P$37, JP4.P$4, JP4.P$44, JP4.P$64, JP4.POWER2
- net GPIO_2: now also JP1.P$2, JP2.P$2, JP3.P$2, JP4.P$2; no longer JP1.P$11, JP2.P$11, JP3.P$11, JP4.P$11
- net MISO: now also JP1.P$72, JP2.P$72, JP3.P$72, JP4.P$72; no longer JP1.P$51, JP2.P$51, JP3.P$51, JP4.P$51
- net MOSI: now also JP1.P$71, JP2.P$71, JP3.P$71, JP4.P$71; no longer JP1.P$50, JP2.P$50, JP3.P$50, JP4.P$50
- net PWM_0: now also JP1.P$31, JP2.P$31, JP3.P$31, JP4.P$31; no longer JP1.P$7, JP2.P$7, JP3.P$7, JP4.P$7
- net PWM_1: now also JP1.P$26, JP2.P$26, JP3.P$26, JP4.P$26; no longer JP1.P$8, JP2.P$8, JP3.P$8, JP4.P$8
- net SPI_CLK: now also JP1.P$70, JP2.P$70, JP3.P$70, JP4.P$70; no longer JP1.P$49, JP2.P$49, JP3.P$49, JP4.P$49
- net USB_1_P: now also JP1.P$41; no longer JP1.P$20
- net USB_2_P: now also JP2.P$41; no longer JP2.P$20
- net USB_3_P: now also JP3.P$41; no longer JP3.P$20
- net USB_4_P: now also JP4.P$41; no longer JP4.P$20
- net V_BATT: now also JP1.POWER2, JP2.POWER2, JP3.POWER2, JP4.POWER2; no longer JP1.POWER1, JP2.POWER1, JP3.POWER1, JP4.POWER1
Other:
- moved on the sheet: JP2, JP3, JP4
