File: Project QUBO/eagleDesigns/backplane/version2/backplane_v4.sch (EAGLE design)
At the start: 302 parts, among them U1 TUSB2077ALQFP

Commit message: 
Parts:
- added R67, R68, R72: 1.5k, resistor:R-US_R0805
Connections:
- net AHRS_USB_M renamed AHRS_USB_N
- net DVL_USB_M renamed DVL_USB_N
- net HUB_USB_M renamed HUB_USB_N
- net IMU_USB_M renamed IMU_USB_N
- removed net EXT_USB_M: 5.7.P$1, R34.2, R47.1, U$5.I/O_2
- removed net N$52: DVL_USB_HUB.XTALOUT
- new net EXT_USB_N: 5.7.P$5, R34.2, R47.1, U$5.I/O_2
- net 3V3: now also R67.2, R68.2, R72.2
- net ACT_SCL: now also 5.4.P$1; no longer 5.4.P$5
- net ACT_SDA: now also 5.5.P$1; no longer 5.5.P$5
- net BATT1_SCL: now also 5.4.P$2; no longer 5.4.P$4
- net BATT1_SDA: now also 5.5.P$2; no longer 5.5.P$4
- net CANH: now also 5.3.P$5; no longer 5.3.P$3
- net DVL_HCTS: now also 5.6.P$2; no longer 5.6.P$4
- net DVL_HRX: now also 5.6.P$5; no longer 5.6.P$1
- net DVL_HTX: now also 5.6.P$4; no longer 5.6.P$2
- net DVL_SCTS: now also 5.7.P$1; no longer 5.7.P$5
- net DVL_SRTS: now also 5.5.P$5; no longer 5.5.P$1
- net DVL_SRX: now also 5.6.P$1; no longer 5.6.P$5
- net DVL_STX: now also 5.4.P$5; no longer 5.4.P$1
- net EXT_SDA: now also 5.3.P$3; no longer 5.3.P$1
- net EXT_USB_5V: now also 5.7.P$2; no longer 5.7.P$4
- net EXT_USB_P: now also 5.7.P$4; no longer 5.7.P$2
- net GND: now also 5.2.P$1, 5.3.P$1; no longer 5.2.P$5, 5.3.P$5
- net HUB_USB_P: now also R72.1
- net N$27: now also R67.1
- net N$38: now also R68.1
- net RTS_MD: now also 5.2.P$2; no longer 5.2.P$4
- net RX_MD: now also 5.2.P$5; no longer 5.2.P$1
- net SHORE_SCL: now also 5.4.P$4; no longer 5.4.P$2
- net SHORE_SDA: now also 5.5.P$4; no longer 5.5.P$2
- net TX_MD: now also 5.2.P$4; no longer 5.2.P$2
Other:
- moved on the sheet: R61, U$49, U$73
