File: Project QUBO/eagleDesigns/backplane/version2/backplane_v4.brd (EAGLE design)
At the start: 141 x 154 mm, 305 parts, among them U1 TUSB2077ALQFP

Commit message: 
Parts:
- moved U$38 160.0 mm to (-77.9, 80.9), turned to 270 degrees
- moved U$39 141.3 mm to (-69.4, 24.1), turned to 270 degrees
- moved U$40 139.7 mm to (-78.2, 36.4), turned to 270 degrees
- moved U$50 128.2 mm to (-76.4, 64.5), turned to 270 degrees
- moved BATTERY-MUX 118.8 mm to (-76.9, 51.3)
- moved G1 110.1 mm to (-88.6, 97.5)
- moved U$13 101.1 mm to (-117.6, -11.9)
- moved U1 69.2 mm to (-55.3, 99.4)
- moved U$33 67.2 mm to (-36.1, 109.7)
- moved DVL_HOST_FTDI 57.7 mm to (-47.6, 70.4)
- moved U$37 57.1 mm to (-52.0, 41.7)
- moved DVL_USB_HUB 55.4 mm to (-26.4, 103.1)
- moved DVL_SLAVE_FTDI 54.4 mm to (-28.8, 79.2)
- moved DVL_TTL-TO-RS232 48.1 mm to (-32.3, 41.4)
- moved U$1 38.7 mm to (-20.3, 114.3)
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Connections:
- net ACT_SCL: now also 5.4.P$1, 5.4.P$2; no longer 5.4.P$10, 5.4.P$9
- net ACT_SDA: now also 5.5.P$1, 5.5.P$2; no longer 5.5.P$10, 5.5.P$9
- net BATT1_SCL: now also 5.4.P$3, 5.4.P$4; no longer 5.4.P$7, 5.4.P$8
- net BATT1_SDA: now also 5.5.P$3, 5.5.P$4; no longer 5.5.P$7, 5.5.P$8
- net CANH: now also 5.3.P$10, 5.3.P$9; no longer 5.3.P$5, 5.3.P$6
- net DVL_HCTS: now also 5.6.P$3, 5.6.P$4; no longer 5.6.P$7, 5.6.P$8
- net DVL_HRX: now also 5.6.P$10, 5.6.P$9; no longer 5.6.P$1, 5.6.P$2
- net DVL_HTX: now also 5.6.P$7, 5.6.P$8; no longer 5.6.P$3, 5.6.P$4
- net DVL_SCTS: now also 5.7.P$1, 5.7.P$2; no longer 5.7.P$10, 5.7.P$9
- net DVL_SRTS: now also 5.5.P$10, 5.5.P$9; no longer 5.5.P$1, 5.5.P$2
- net DVL_SRX: now also 5.6.P$1, 5.6.P$2; no longer 5.6.P$10, 5.6.P$9
- net DVL_STX: now also 5.4.P$10, 5.4.P$9; no longer 5.4.P$1, 5.4.P$2
- net EXT_SDA: now also 5.3.P$5, 5.3.P$6; no longer 5.3.P$1, 5.3.P$2
- net EXT_USB_5V: now also 5.7.P$3, 5.7.P$4; no longer 5.7.P$7, 5.7.P$8
- net EXT_USB_N: now also 5.7.P$10, 5.7.P$9; no longer 5.7.P$1, 5.7.P$2
- net EXT_USB_P: now also 5.7.P$7, 5.7.P$8; no longer 5.7.P$3, 5.7.P$4
- net GND: now also 5.2.P$1, 5.2.P$2, 5.3.P$1, 5.3.P$2; no longer 5.2.P$10, 5.2.P$9, 5.3.P$10, 5.3.P$9
- net RTS_MD: now also 5.2.P$3, 5.2.P$4; no longer 5.2.P$7, 5.2.P$8
- net RX_MD: now also 5.2.P$10, 5.2.P$9; no longer 5.2.P$1, 5.2.P$2
- net SHORE_SCL: now also 5.4.P$7, 5.4.P$8; no longer 5.4.P$3, 5.4.P$4
- net SHORE_SDA: now also 5.5.P$7, 5.5.P$8; no longer 5.5.P$3, 5.5.P$4
- net TX_MD: now also 5.2.P$7, 5.2.P$8; no longer 5.2.P$3, 5.2.P$4
Routing:
- net 12V: track 80.7 -> 137.3 mm
- net 5V: track 80.7 -> 122.5 mm
- net GND: track 0.00 -> 10.2 mm
- net RX_MD: track 5.08 -> 0.00 mm
- net SHORE_SDA: track 0.00 -> 5.08 mm
- net EXT_USB_P: track 0.00 -> 5.08 mm
- net EXT_USB_N: track 0.00 -> 5.08 mm
- net EXT_USB_5V: track 0.00 -> 5.08 mm
- net EXT_SDA: track 0.00 -> 5.08 mm
- net EXT_SCL: track 0.00 -> 5.08 mm
- net DVL_SRTS: track 0.00 -> 5.08 mm
- net DVL_SCTS: track 0.00 -> 5.08 mm
- net CANL: track 0.00 -> 5.08 mm
- net BATT2_SDA: track 0.00 -> 5.08 mm
- net BATT1_SDA: track 0.00 -> 5.08 mm
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