File: Project QUBO/eagleDesigns/Jr Support/Charging/charging_block.sch (EAGLE design)
At the start: 115 parts

Commit message: 
Parts:
- U$39, U$5: value SBR2065 -> (none); device diode:SBR2065 -> diode:SCHOTTKY-DIODESOD-106
Connections:
- net V_CHARGE1 renamed N$56
- net V_CHARGE2 renamed N$44
- removed net N$35: R18.1, U$11.G
- new net N$38: R16.1, U$1.!FASTCHG!, U$10.G
- net N$32: now also R18.1, U$1.!FULLCHG!, U$11.G; no longer R16.1, U$10.G
- net N$36: now also U$1.!FAULT!
Other:
- moved on the sheet: BATT1_CHARGE, C11, R4, R6, U$15, U$16, U$22
Changed lines of the file:
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@@
 <part name="R29" library="resistor" deviceset="R-US_" device="R0805" value="100m"/>
 <part name="U$38" library="resistor" deviceset="DUAL-L" device=""/>
-<part name="U$39" library="diode" deviceset="SBR2065" device=""/>
+<part name="U$39" library="diode" deviceset="SCHOTTKY-DIODE" device="SOD-106"/>
 <part name="D1" library="diode" deviceset="DIODE-" device="SOD123"/>
 <part name="U$40" library="vishay" deviceset="NTCLE201E3" device=""/>
@@
 <part name="C19" library="resistor" deviceset="C-US" device="C0805" value="100u,&lt;50mO"/>
 <part name="R7" library="resistor" deviceset="R-US_" device="R0805" value="100m"/>
-<part name="U$5" library="diode" deviceset="SBR2065" device=""/>
+<part name="U$5" library="diode" deviceset="SCHOTTKY-DIODE" device="SOD-106"/>
 <part name="D2" library="diode" deviceset="DIODE-" device="SOD123"/>
 <part name="U$6" library="vishay" deviceset="NTCLE201E3" device=""/>
@@
 <instance part="V_OUT" gate="G$1" x="302.26" y="137.16" rot="MR0"/>
 <instance part="U$21" gate="G$1" x="312.42" y="137.16"/>
-<instance part="BATT1_CHARGE" gate="G$1" x="170.18" y="-58.42" rot="MR270"/>
-<instance part="U$15" gate="G$1" x="170.18" y="-40.64" rot="MR270"/>
-<instance part="U$16" gate="G$1" x="165.1" y="-35.56"/>
-<instance part="R4" gate="G$1" x="144.78" y="-38.1" rot="MR0"/>
-<instance part="C11" gate="G$1" x="154.94" y="-33.02" rot="MR180"/>
-<instance part="U$22" gate="G$1" x="134.62" y="-25.4" rot="MR270"/>
-<instance part="R6" gate="G$1" x="134.62" y="-43.18" rot="MR90"/>
+<instance part="BATT1_CHARGE" gate="G$1" x="167.64" y="-58.42" rot="MR270"/>
+<instance part="U$15" gate="G$1" x="167.64" y="-40.64" rot="MR270"/>
+<instance part="U$16" gate="G$1" x="162.56" y="-35.56"/>
+<instance part="R4" gate="G$1" x="142.24" y="-38.1" rot="MR0"/>
+<instance part="C11" gate="G$1" x="152.4" y="-33.02" rot="MR180"/>
+<instance part="U$22" gate="G$1" x="132.08" y="-25.4" rot="MR270"/>
+<instance part="R6" gate="G$1" x="132.08" y="-43.18" rot="MR90"/>
 <instance part="BATT2_CHARGE" gate="G$1" x="218.44" y="-58.42" rot="R270"/>
 <instance part="U$13" gate="G$1" x="218.44" y="-40.64" rot="R270"/>
@@
 <segment>
 <pinref part="BATT1_CHARGE" gate="G$1" pin="P$2"/>
-<wire x1="172.72" y1="-50.8" x2="172.72" y2="-40.64" width="0.1524" layer="91"/>
-<wire x1="172.72" y1="-40.64" x2="180.34" y2="-40.64" width="0.1524" layer="91"/>
-<label x="177.8" y="-40.64" size="1.778" layer="95" rot="MR180"/>
+<wire x1="170.18" y1="-50.8" x2="170.18" y2="-40.64" width="0.1524" layer="91"/>
+<wire x1="170.18" y1="-40.64" x2="177.8" y2="-40.64" width="0.1524" layer="91"/>
+<label x="175.26" y="-40.64" size="1.778" layer="95" rot="MR180"/>
 <pinref part="U$15" gate="G$1" pin="A"/>
-<junction x="172.72" y="-40.64"/>
+<junction x="170.18" y="-40.64"/>
 </segment>
 <segment>
 <pinref part="U$22" gate="G$1" pin="P$1"/>
 <pinref part="C11" gate="G$1" pin="2"/>
-<wire x1="134.62" y1="-17.78" x2="154.94" y2="-17.78" width="0.1524" layer="91"/>
-<wire x1="154.94" y1="-17.78" x2="154.94" y2="-27.94" width="0.1524" layer="91"/>
-<label x="149.86" y="-17.78" size="1.778" layer="95" rot="MR180"/>
+<wire x1="132.08" y1="-17.78" x2="152.4" y2="-17.78" width="0.1524" layer="91"/>
+<wire x1="152.4" y1="-17.78" x2="152.4" y2="-27.94" width="0.1524" layer="91"/>
+<label x="147.32" y="-17.78" size="1.778" layer="95" rot="MR180"/>
 </segment>
 <segment>
@@
 <wire x1="142.24" y1="96.52" x2="137.16" y2="96.52" width="0.1524" layer="91"/>
 <wire x1="137.16" y1="96.52" x2="137.16" y2="127" width="0.1524" layer="91"/>
+<junction x="137.16" y="96.52"/>
 </segment>
 </net>
@@
 </segment>
 </net>
-<net name="N$32" class="0">
-<segment>
-<pinref part="U$10" gate="G$1" pin="G"/>
-<pinref part="R16" gate="G$1" pin="1"/>
-<wire x1="386.08" y1="7.62" x2="378.46" y2="7.62" width="0.1524" layer="91"/>
-<wire x1="378.46" y1="7.62" x2="340.36" y2="7.62" width="0.1524" layer="91"/>
-<wire x1="340.36" y1="7.62" x2="340.36" y2="10.16" width="0.1524" layer="91"/>
-<junction x="378.46" y="7.62"/>
-<wire x1="340.36" y1="10.16" x2="312.42" y2="10.16" width="0.1524" layer="91"/>
-</segment>
-</net>
 <net name="N$33" class="0">
 <segment>
@@
 <pinref part="U$11" gate="G$1" pin="D"/>
 <wire x1="386.08" y1="-38.1" x2="386.08" y2="-30.48" width="0.1524" layer="91"/>
-</segment>
-</net>
-<net name="N$35" class="0">
-<segment>
-<pinref part="U$11" gate="G$1" pin="G"/>
-<pinref part="R18" gate="G$1" pin="1"/>
-<wire x1="373.38" y1="-20.32" x2="365.76" y2="-20.32" width="0.1524" layer="91"/>
-<wire x1="312.42" y1="7.62" x2="337.82" y2="7.62" width="0.1524" layer="91"/>
-<wire x1="337.82" y1="7.62" x2="337.82" y2="-20.32" width="0.1524" layer="91"/>
-<wire x1="337.82" y1="-20.32" x2="365.76" y2="-20.32" width="0.1524" layer="91"/>
-<junction x="365.76" y="-20.32"/>
-</segment>
-</net>
-<net name="N$38" class="0">
-<segment>
-<wire x1="312.42" y1="-48.26" x2="312.42" y2="5.08" width="0.1524" layer="91"/>
 </segment>
 </net>
@@
 <pinref part="R20" gate="G$1" pin="1"/>
 <wire x1="360.68" y1="-48.26" x2="353.06" y2="-48.26" width="0.1524" layer="91"/>
-<wire x1="353.06" y1="-48.26" x2="312.42" y2="-48.26" width="0.1524" layer="91"/>
+<pinref part="U$1" gate="G$1" pin="!FAULT!"/>
+<wire x1="312.42" y1="5.08" x2="312.42" y2="-48.26" width="0.1524" layer="91"/>
+<wire x1="312.42" y1="-48.26" x2="353.06" y2="-48.26" width="0.1524" layer="91"/>
 <junction x="353.06" y="-48.26"/>
 </segment>
@@
 <pinref part="BATT1_CHARGE" gate="G$1" pin="P$1"/>
 <pinref part="U$15" gate="G$1" pin="C"/>
-<wire x1="167.64" y1="-50.8" x2="167.64" y2="-40.64" width="0.1524" layer="91"/>
+<wire x1="165.1" y1="-50.8" x2="165.1" y2="-40.64" width="0.1524" layer="91"/>
 <pinref part="U$16" gate="G$1" pin="D"/>
-<junction x="167.64" y="-40.64"/>
+<junction x="165.1" y="-40.64"/>
 <pinref part="R6" gate="G$1" pin="1"/>
-<wire x1="134.62" y1="-48.26" x2="134.62" y2="-50.8" width="0.1524" layer="91"/>
-<wire x1="134.62" y1="-50.8" x2="167.64" y2="-50.8" width="0.1524" layer="91"/>
-<junction x="167.64" y="-50.8"/>
+<wire x1="132.08" y1="-48.26" x2="132.08" y2="-50.8" width="0.1524" layer="91"/>
+<wire x1="132.08" y1="-50.8" x2="165.1" y2="-50.8" width="0.1524" layer="91"/>
+<junction x="165.1" y="-50.8"/>
 </segment>
 </net>
@@
 <pinref part="C11" gate="G$1" pin="1"/>
 <pinref part="R4" gate="G$1" pin="1"/>
-<wire x1="154.94" y1="-35.56" x2="154.94" y2="-38.1" width="0.1524" layer="91"/>
-<wire x1="154.94" y1="-38.1" x2="149.86" y2="-38.1" width="0.1524" layer="91"/>
+<wire x1="152.4" y1="-35.56" x2="152.4" y2="-38.1" width="0.1524" layer="91"/>
+<wire x1="152.4" y1="-38.1" x2="147.32" y2="-38.1" width="0.1524" layer="91"/>
 <pinref part="U$16" gate="G$1" pin="G"/>
-<wire x1="154.94" y1="-38.1" x2="160.02" y2="-38.1" width="0.1524" layer="91"/>
-<junction x="154.94" y="-38.1"/>
+<wire x1="152.4" y1="-38.1" x2="157.48" y2="-38.1" width="0.1524" layer="91"/>
+<junction x="152.4" y="-38.1"/>
 </segment>
 </net>
@@
 <pinref part="R4" gate="G$1" pin="2"/>
 <pinref part="U$22" gate="G$1" pin="P$2"/>
-<wire x1="139.7" y1="-38.1" x2="134.62" y2="-38.1" width="0.1524" layer="91"/>
-<wire x1="134.62" y1="-38.1" x2="134.62" y2="-33.02" width="0.1524" layer="91"/>
+<wire x1="137.16" y1="-38.1" x2="132.08" y2="-38.1" width="0.1524" layer="91"/>
+<wire x1="132.08" y1="-38.1" x2="132.08" y2="-33.02" width="0.1524" layer="91"/>
 <pinref part="R6" gate="G$1" pin="2"/>
-<junction x="134.62" y="-38.1"/>
-</segment>
-</net>
-<net name="V_CHARGE1" class="0">
-<segment>
-<pinref part="U$16" gate="G$1" pin="S"/>
-<pinref part="U$17" gate="G$1" pin="P$1"/>
-<wire x1="165.1" y1="10.16" x2="167.64" y2="10.16" width="0.1524" layer="91"/>
-<label x="170.18" y="-7.62" size="1.778" layer="95"/>
-<wire x1="167.64" y1="-30.48" x2="167.64" y2="10.16" width="0.1524" layer="91"/>
+<junction x="132.08" y="-38.1"/>
 </segment>
 </net>
@@
 </segment>
 </net>
-<net name="V_CHARGE2" class="0">
-<segment>
+<net name="N$44" class="0">
+<segment>
+<pinref part="U$23" gate="G$1" pin="S"/>
 <pinref part="U$18" gate="G$1" pin="P$1"/>
-<label x="205.74" y="-7.62" size="1.778" layer="95"/>
-<wire x1="220.98" y1="-17.78" x2="220.98" y2="10.16" width="0.1524" layer="91"/>
-</segment>
-<segment>
-<pinref part="U$23" gate="G$1" pin="S"/>
-<wire x1="220.98" y1="-30.48" x2="220.98" y2="-17.78" width="0.1524" layer="91"/>
+<wire x1="220.98" y1="-30.48" x2="220.98" y2="10.16" width="0.1524" layer="91"/>
+</segment>
+</net>
+<net name="N$56" class="0">
+<segment>
+<pinref part="U$16" gate="G$1" pin="S"/>
+<pinref part="U$17" gate="G$1" pin="P$1"/>
+<wire x1="165.1" y1="-30.48" x2="165.1" y2="10.16" width="0.1524" layer="91"/>
+</segment>
+</net>
+<net name="N$38" class="0">
+<segment>
+<pinref part="R16" gate="G$1" pin="1"/>
+<pinref part="U$10" gate="G$1" pin="G"/>
+<wire x1="386.08" y1="7.62" x2="378.46" y2="7.62" width="0.1524" layer="91"/>
+<pinref part="U$1" gate="G$1" pin="!FASTCHG!"/>
+<wire x1="312.42" y1="10.16" x2="340.36" y2="10.16" width="0.1524" layer="91"/>
+<wire x1="340.36" y1="10.16" x2="340.36" y2="7.62" width="0.1524" layer="91"/>
+<wire x1="340.36" y1="7.62" x2="378.46" y2="7.62" width="0.1524" layer="91"/>
+<junction x="378.46" y="7.62"/>
+</segment>
+</net>
+<net name="N$32" class="0">
+<segment>
+<pinref part="R18" gate="G$1" pin="1"/>
+<pinref part="U$11" gate="G$1" pin="G"/>
+<wire x1="373.38" y1="-20.32" x2="365.76" y2="-20.32" width="0.1524" layer="91"/>
+<pinref part="U$1" gate="G$1" pin="!FULLCHG!"/>
+<wire x1="312.42" y1="7.62" x2="337.82" y2="7.62" width="0.1524" layer="91"/>
+<wire x1="337.82" y1="7.62" x2="337.82" y2="-20.32" width="0.1524" layer="91"/>
+<wire x1="337.82" y1="-20.32" x2="365.76" y2="-20.32" width="0.1524" layer="91"/>
+<junction x="365.76" y="-20.32"/>
 </segment>
 </net>
@@
 </sheet>
 </sheets>
+<errors>
+</errors>
 </schematic>
 </drawing>

Commit message: 
Parts:
- removed U$38: (no value), resistor:DUAL-L
- added L1, L2: 10u, resistor:L-USL6100
- added LED7, LED8: Green, led:LEDCHIP-LED0805
- added R28, R33: 330, resistor:R-US_R0805
Connections:
- new net N$35: LED7.A, R28.1
- new net N$57: LED8.A, R33.1
- net GND: now also LED7.C, LED8.C
- net N$17: now also L2.1; no longer U$38.P$2
- net N$20: now also L2.2; no longer U$38.P$4
- net N$77: now also L1.2; no longer U$38.P$3
- net N$81: now also L1.1; no longer U$38.P$1
Changed lines of the file:
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@@
 <part name="C84" library="resistor" deviceset="C-US" device="C0805" value="100u,&lt;50mO"/>
 <part name="R29" library="resistor" deviceset="R-US_" device="R0805" value="100m"/>
-<part name="U$38" library="resistor" deviceset="DUAL-L" device=""/>
 <part name="U$39" library="diode" deviceset="SCHOTTKY-DIODE" device="SOD-106"/>
 <part name="D1" library="diode" deviceset="DIODE-" device="SOD123"/>
@@
 <part name="U$24" library="switches" deviceset="GPTS203212B" device=""/>
 <part name="R27" library="resistor" deviceset="R-US_" device="R0805" value="4.3k"/>
+<part name="LED7" library="led" deviceset="LED" device="CHIP-LED0805" value="Green"/>
+<part name="R28" library="resistor" deviceset="R-US_" device="R0805" value="330"/>
+<part name="LED8" library="led" deviceset="LED" device="CHIP-LED0805" value="Green"/>
+<part name="R33" library="resistor" deviceset="R-US_" device="R0805" value="330"/>
+<part name="L1" library="resistor" deviceset="L-US" device="L6100" value="10u"/>
+<part name="L2" library="resistor" deviceset="L-US" device="L6100" value="10u"/>
 </parts>
 <sheets>
@@
 <instance part="C84" gate="G$1" x="137.16" y="7.62"/>
 <instance part="R29" gate="G$1" x="144.78" y="15.24" rot="R90"/>
-<instance part="U$38" gate="G$1" x="193.04" y="40.64"/>
 <instance part="U$39" gate="G$1" x="30.48" y="81.28"/>
 <instance part="D1" gate="G$1" x="109.22" y="40.64" rot="R90"/>
@@
 <instance part="U$24" gate="G$1" x="254" y="-25.4" rot="R270"/>
 <instance part="R27" gate="G$1" x="254" y="-43.18" rot="R90"/>
+<instance part="LED7" gate="G$1" x="236.22" y="119.38"/>
+<instance part="R28" gate="G$1" x="236.22" y="127" rot="R90"/>
+<instance part="LED8" gate="G$1" x="193.04" y="83.82"/>
+<instance part="R33" gate="G$1" x="193.04" y="91.44" rot="R90"/>
+<instance part="L1" gate="G$1" x="137.16" y="38.1"/>
+<instance part="L2" gate="G$1" x="248.92" y="38.1"/>
 </instances>
 <busses>
@@
 <label x="238.76" y="-17.78" size="1.778" layer="95" rot="R180"/>
 </segment>
+<segment>
+<pinref part="LED8" gate="G$1" pin="C"/>
+<wire x1="193.04" y1="78.74" x2="193.04" y2="73.66" width="0.1524" layer="91"/>
+<label x="193.04" y="73.66" size="1.778" layer="95"/>
+</segment>
+<segment>
+<pinref part="LED7" gate="G$1" pin="C"/>
+<wire x1="236.22" y1="114.3" x2="236.22" y2="109.22" width="0.1524" layer="91"/>
+<label x="236.22" y="109.22" size="1.778" layer="95"/>
+</segment>
 </net>
 <net name="V_BATT1" class="0">
@@
 <wire x1="121.92" y1="38.1" x2="121.92" y2="45.72" width="0.1524" layer="91"/>
 <wire x1="121.92" y1="45.72" x2="121.92" y2="53.34" width="0.1524" layer="91"/>
-<wire x1="121.92" y1="45.72" x2="182.88" y2="45.72" width="0.1524" layer="91"/>
+<wire x1="121.92" y1="45.72" x2="137.16" y2="45.72" width="0.1524" layer="91"/>
 <junction x="121.92" y="45.72"/>
-<pinref part="U$38" gate="G$1" pin="P$1"/>
+<pinref part="L1" gate="G$1" pin="1"/>
 </segment>
 </net>
@@
 <wire x1="137.16" y1="20.32" x2="144.78" y2="20.32" width="0.1524" layer="91"/>
 <junction x="137.16" y="20.32"/>
-<pinref part="U$38" gate="G$1" pin="P$3"/>
-<wire x1="137.16" y1="20.32" x2="137.16" y2="35.56" width="0.1524" layer="91"/>
-<wire x1="137.16" y1="35.56" x2="182.88" y2="35.56" width="0.1524" layer="91"/>
+<wire x1="137.16" y1="20.32" x2="137.16" y2="30.48" width="0.1524" layer="91"/>
+<pinref part="L1" gate="G$1" pin="2"/>
 </segment>
 </net>
@@
 <pinref part="U$40" gate="G$1" pin="1"/>
 <wire x1="109.22" y1="-5.08" x2="119.38" y2="-5.08" width="0.1524" layer="91"/>
-</segment>
-</net>
-<net name="N$1" class="0">
-<segment>
-<pinref part="R1" gate="G$1" pin="2"/>
-<pinref part="R2" gate="G$1" pin="2"/>
-<pinref part="U$1" gate="G$1" pin="VADJ"/>
-<wire x1="312.42" y1="50.8" x2="327.66" y2="50.8" width="0.1524" layer="91"/>
-<junction x="327.66" y="50.8"/>
-<wire x1="327.66" y1="50.8" x2="325.12" y2="50.8" width="0.1524" layer="91"/>
 </segment>
 </net>
@@
 </segment>
 </net>
-<net name="N$6" class="0">
-<segment>
-<pinref part="U$1" gate="G$1" pin="CCV"/>
-<pinref part="C6" gate="G$1" pin="1"/>
-<wire x1="312.42" y1="43.18" x2="327.66" y2="43.18" width="0.1524" layer="91"/>
-<pinref part="R3" gate="G$1" pin="2"/>
-<junction x="327.66" y="43.18"/>
-<wire x1="327.66" y1="43.18" x2="322.58" y2="43.18" width="0.1524" layer="91"/>
-</segment>
-</net>
 <net name="N$7" class="0">
 <segment>
@@
 <wire x1="264.16" y1="45.72" x2="264.16" y2="53.34" width="0.1524" layer="91"/>
 <junction x="264.16" y="45.72"/>
-<pinref part="U$38" gate="G$1" pin="P$2"/>
-<wire x1="264.16" y1="45.72" x2="203.2" y2="45.72" width="0.1524" layer="91"/>
+<wire x1="264.16" y1="45.72" x2="248.92" y2="45.72" width="0.1524" layer="91"/>
+<pinref part="L2" gate="G$1" pin="1"/>
 </segment>
 </net>
@@
 <wire x1="248.92" y1="20.32" x2="241.3" y2="20.32" width="0.1524" layer="91"/>
 <junction x="248.92" y="20.32"/>
-<wire x1="248.92" y1="35.56" x2="248.92" y2="20.32" width="0.1524" layer="91"/>
-<pinref part="U$38" gate="G$1" pin="P$4"/>
-<wire x1="203.2" y1="35.56" x2="248.92" y2="35.56" width="0.1524" layer="91"/>
+<wire x1="248.92" y1="30.48" x2="248.92" y2="20.32" width="0.1524" layer="91"/>
+<pinref part="L2" gate="G$1" pin="2"/>
 </segment>
 </net>
@@
 </segment>
 </net>
+<net name="N$35" class="0">
+<segment>
+<pinref part="LED7" gate="G$1" pin="A"/>
+<pinref part="R28" gate="G$1" pin="1"/>
+</segment>
+</net>
+<net name="N$57" class="0">
+<segment>
+<pinref part="LED8" gate="G$1" pin="A"/>
+<pinref part="R33" gate="G$1" pin="1"/>
+</segment>
+</net>
+<net name="N$1" class="0">
+<segment>
+<pinref part="U$1" gate="G$1" pin="CCV"/>
+<pinref part="C6" gate="G$1" pin="1"/>
+<wire x1="312.42" y1="43.18" x2="322.58" y2="43.18" width="0.1524" layer="91"/>
+<pinref part="R3" gate="G$1" pin="2"/>
+<wire x1="322.58" y1="43.18" x2="327.66" y2="43.18" width="0.1524" layer="91"/>
+<junction x="322.58" y="43.18"/>
+</segment>
+</net>
+<net name="N$6" class="0">
+<segment>
+<pinref part="R2" gate="G$1" pin="2"/>
+<pinref part="R1" gate="G$1" pin="2"/>
+<wire x1="327.66" y1="50.8" x2="325.12" y2="50.8" width="0.1524" layer="91"/>
+<pinref part="U$1" gate="G$1" pin="VADJ"/>
+<wire x1="325.12" y1="50.8" x2="312.42" y2="50.8" width="0.1524" layer="91"/>
+<junction x="325.12" y="50.8"/>
+</segment>
+</net>

Commit message: Charging board layout, rev. 1
Parts:
- added R35, R36, R37: 0, resistor:R-US_R0805
- C19: value 100u,<50mO -> 120uF; device resistor:C-USC0805 -> resistor:CPOL-USE3.5-8
- C84: value 100u,<50mO -> 120u; device resistor:C-USC0805 -> resistor:CPOL-USE3.5-8
- R28: value 330 -> 1.5k
Connections:
- net N$11 renamed BATT1_P
- net N$15 renamed DLO_2
- net N$16 renamed DHI_2
- net N$17 renamed L-IN_2
- net N$18 renamed PGND_2
- net N$20 renamed CS_2
- net N$21 renamed THM_2
- net N$42 renamed DCIN_2
- net N$43 renamed BATT2_P
- net N$45 renamed VIN
- net N$46 renamed FET-G_1
- net N$56 renamed FET-D_1
- net N$77 renamed CS_1
- removed net N$48: C60.2, ON.P$2, U$56.GND, U$58.A
- removed net V_BATT1: C83.1, C84.1, R29.1, R34.1, U$17.P$2, U$33.BATT
- removed net V_BATT2: C18.1, C19.1, R5.1, R7.1, U$1.BATT, U$18.P$2
- new net BATT1_M: BATT1_CHARGE.P$2, R35.1, R37.1, U$15.A, U$40.2
- new net BATT2_M: BATT2_CHARGE.P$2, R36.2, U$13.A, U$6.2
- new net BATT_1: C83.1, C84.+, R29.1, R34.1, U$17.P$2, U$33.BATT
- new net BATT_2: C18.1, C19.+, R5.1, R7.1, U$1.BATT, U$18.P$2
- net !SHDN!: now also R33.2
- net GND: now also C19.-, C60.2, C84.-, ON.P$2, R35.2, R36.1, R37.2, U$56.GND, U$58.A; no longer BATT1_CHARGE.P$2, BATT2_CHARGE.P$2, C19.2, C84.2, U$13.A, U$15.A, U$40.2, U$6.2
- net V_SHORE: now also R28.2

Commit message: Charging board version 1 - completed
Parts:
- B1-HFET, U$2, U$3, U$37: value (none) -> FDMC8360LET40PWR33
- L1, L2: value 10u -> 10uH
- LED1, LED4: value Green -> FASTCHG
- LED2, LED5: value Green -> FULLCHG
- LED3, LED6: value Red -> FAULT
- LED7: value Green -> Shore Power
- LED8: value Green -> CHARGING
- renumbered AUDIO to BUZZER, AUDIO1 to BUZZER2, BATT1_CHARGE to BATT1_IN, BATT2_CHARGE to BATT2_IN, ON to CHARGING-SWITCH, U$13 to 24V-TVS_3, U$15 to 24V-TVS_2, U$17 to BATT1_FUSE, U$18 to BATT2_FUSE, U$20 to INPUT-SWITCH, U$21 to 24V-TVS_OUT, U$22 to BATT1_SWITCH, U$24 to BATT2_SWITCH, U$33 to BATT1_IC, U$34 to B1-HFET, U$39 to B1-ZENER, U$4 to 24V-TVS_1, U$58 to 5V-TVS_1, VIN to SHORE_IN, V_OUT to SHORE_OUT
