File: Project QUBO/eagleDesigns/Jr Support/Charging/charging_block_v2.brd (EAGLE design)
At the start: 54.6 x 93 mm, 73 parts, among them U56 74LVC1G14, U57 NCP1117, U7 SSM3J353F, U8 SSM3J353F, U9 SSM3J353F

Commit message: 
Parts:
- C67: value 2.2u -> 0.1u
- R1: value 2-3k -> 2.1k
- R30, R31: value ~50k -> 50k
Changed lines of the file:
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@@
 <attribute name="VALUE" x="14.351" y="60.071" size="0.8128" layer="27" ratio="17" rot="R90"/>
 </element>
-<element name="C67" library="resistor" package="C0805" value="2.2u" x="16.51" y="60.96" smashed="yes" rot="R90">
+<element name="C67" library="resistor" package="C0805" value="0.1u" x="16.51" y="60.96" smashed="yes" rot="R90">
 <attribute name="NAME" x="17.399" y="63.754" size="0.8128" layer="25" ratio="17" rot="R180"/>
 <attribute name="VALUE" x="18.796" y="60.071" size="0.8128" layer="27" ratio="17" rot="R90"/>
@@
 <attribute name="VALUE" x="53.975" y="37.973" size="0.8128" layer="27" ratio="17" rot="R90"/>
 </element>
-<element name="R30" library="resistor" package="R0805" value="~50k" x="13.208" y="55.499" smashed="yes" rot="R270">
+<element name="R30" library="resistor" package="R0805" value="50k" x="13.208" y="55.499" smashed="yes" rot="R270">
 <attribute name="NAME" x="12.319" y="57.404" size="0.8128" layer="25" ratio="17"/>
 <attribute name="VALUE" x="10.922" y="56.261" size="0.8128" layer="27" ratio="17" rot="R270"/>
 </element>
-<element name="R31" library="resistor" package="R0805" value="~50k" x="10.16" y="55.118" smashed="yes">
+<element name="R31" library="resistor" package="R0805" value="50k" x="10.16" y="55.118" smashed="yes">
 <attribute name="NAME" x="8.001" y="53.848" size="0.8128" layer="25" ratio="17" rot="R90"/>
 <attribute name="VALUE" x="9.398" y="52.832" size="0.8128" layer="27" ratio="17"/>
@@
 <attribute name="VALUE" x="6.35" y="18.415" size="0.8128" layer="27" ratio="17" rot="R180"/>
 </element>
-<element name="R1" library="resistor" package="R0805" value="2-3k" x="8.89" y="15.875" smashed="yes">
+<element name="R1" library="resistor" package="R0805" value="2.1k" x="8.89" y="15.875" smashed="yes">
 <attribute name="NAME" x="10.287" y="14.859" size="0.8128" layer="25" ratio="17" rot="R180"/>
 <attribute name="VALUE" x="8.128" y="13.589" size="0.8128" layer="27" ratio="17"/>
