File: Project QUBO/eagleDesigns/Jr Support/Charging/charging_block_v3.brd (EAGLE design)
At the start: 54.6 x 93 mm, 73 parts, among them U56 74LVC1G14, U57 NCP1117, U7 SSM3J353F, U8 SSM3J353F, U9 SSM3J353F

Commit message: 
Parts:
- C67: value 2.2u -> 0.1u
- R1: value 2-3k -> 2.1k
- R30, R31: value ~50k -> 50k
- moved THERM 7.24 mm to (31.8, 39.4)
- moved B1-ZENER 1.27 mm to (21.0, 63.5)
Routing:
- net GND: track 73.3 -> 87.8 mm, vias 29 -> 30
- net BATT1_P: track 16.6 -> 18.9 mm
- net N$49: track 2.22 -> 4.26 mm
- net THM1: track 22.7 -> 24.4 mm, vias 2 -> 1
- net VL_1: track 17.2 -> 18.4 mm
- net DCIN_1: track 7.29 -> 8.33 mm
- net V_SHORE: track 190.1 -> 189.4 mm
