File: Project QUBO/eagleDesigns/Jr Support/Jr Support/jr-support_v4.brd (EAGLE design)
At the start: 203.2 x 127 mm, 207 parts, among them U1 PCA9685

Commit message: updated jr support
Parts:
- removed 12V_REG, 5V_REG: LT8640, linear:QFN18-3X4
- removed 5-TVS_1, 5-TVS_2, 5-TVS_3: BZA408B, diodes:SOT457
- removed 5V_PG: Red, led:CHIP-LED0805
- removed C39, C63: 1u, resistor:C0805
- removed C41: 0.1u, resistor:C0805
- removed C42: 15p, resistor:C0805
- removed L1, L2: 2.2u, resistor:L0740
- removed LED2: RED, led:CHIP-LED0805
- removed R2, R38: 1.2k, resistor:R0805
- removed R3, R40: 50k, resistor:R0805
- removed TVS1, TVS2, TVS3: (no value), diode:SOD-323
- removed U$66: SSM3J353F, transistors:SOT-346-3/S-MINI
- added 2PIN_5, AUDIO, AUDIO1, BATT1_IN, BATT2_IN, SHORE_IN: KK254_VERT_2PIN"", molex:KK254_VERT_2PIN
- added C50: 330 uF, resistor:CKR_D10
- added C51: .1 uF, resistor:C0805
- added CIN1, CIN2, CIN3, CIN4: 2.2 uF, resistor:C1210
- added JP1, JP2: (no value), jumper:JP1
- added JP6: 2_SUPERSABRE, molex:SUPERSABRE_2CIRCUIT
- added LED1, LED3: Red, led:0805
- added LED4: Green, led:CHIPLED_0805
- added LED5, LED8, LED9: Green, led:0805
- added LED6, LED7: Yellow, led:0805
- added PMOS1, PMOS2: SSM3J353F, transistors:SOT-346-3/S-MINI
- added POT, POT1: 10k, resistor:PTV09A-4
- added R12: 5m, resistor:R0805
- added R13: 20.8k, resistor:R0805
- added R19, R28: 8.2k, resistor:R0805
- added R20: 5.1k, resistor:R0805
- added R22: 510, resistor:R0805
- added R26: 10\, resistor:R0805
- added R27: 200k, resistor:R0805
- added R29: 6.8k, resistor:R0805
- added R36, R41, R45, R47: 20k, resistor:R0805
- added R37, R42: 430, resistor:R0805
- added R39, R43, R48, R49: 330, resistor:R0805
- added R44, R46: 1.2k, resistor:R0805
- added R5: 21kO, resistor:RC55
- added R50, R51: 1.5k, resistor:R0805
- added R6: 2.61kO, resistor:RC55
- added R9: 12k, resistor:R0805
- added TEST-PTS, TEST-PTS1: 0, resistor:V526-0
- added U$25, U$41: PTN78060W, texas:PTN78060W
- added U$42, U$43, U$44, U$46, U$47, U$62, U$65: VTVSSOT323, diode:SOT323-R
- added U$48, U$51: LTC4364MSOP, linear:MSOP16
- added U$49, U$50, U$52, U$53: STD95N2LH5, transistors:DPAK
- added U$54, U$63, U$64: VTVSDO-219AB, diode:DO-219AB
- added U$55, U$58: BSS138CT-NDSOT23, transistor-fet:SOT23
- added U$56: 74LVC1G14, NXP:TSSOP5
- added U$57: NCP1117, ONSemi:SOT-223
- added U$60, U$61: TL431DBZ, texas:SOT-23-3
- 2PIN_1, CAMERA1, CAMERA2, ETHERNET, FAN1, FAN2, SW_CPU: value KK254_VERT_2PIN22-29-2021 -> KK254_VERT_2PIN""
- C27: value 10u -> 0.22u
- C28: value 15p -> 22u
- C35: value 22u -> 1u
- C36: value 220u -> 1u; device resistor:C-F80 -> resistor:C0805
- C38: value 1u -> 330 uF; device resistor:C0805 -> resistor:CKR_D10
- C4: value 1u -> 0.22u
- C40: value 10u -> .1 uF
- C61: value 22u -> 10u
- C62: value 220u -> 10u; device resistor:C-F80 -> resistor:C0805
- C65: value 0.1u -> 22u
- JP3: value MPTC-01-80 -> (none); device samtec:MPTC-01-80 -> pinhead:1X02
- R14: value 41.2k -> 51k
- R15: value 1M -> 5m
- R16: value 88.7k -> 10\
- R17: value 41.2k -> 200k
- R23: value 1M -> 51k
- R24: value 243k -> 5.1k
- U$1: value SSM3J353F -> VTVSDO-219AB; device transistors:SOT-346-3/S-MINI -> diode:DO-219AB
- U$10, U$13, U$16, U$21, U$22, U$26, U$28, U$30, U$31, U$32, U$33, U$34, U$38, U$59: value VTVS -> VTVSSOT323; device diode:DO-219AB -> diode:SOT323-R
- moved U$1 1094.6 mm to (-265.4, -1032.5), turned to 0 degrees
- moved JP3 1081.9 mm to (-208.3, -969.0)
- moved C62 1055.0 mm to (-200.7, -1002.0), turned to 0 degrees
- moved R24 1053.6 mm to (-212.1, -995.7), turned to 0 degrees
- moved R17 1053.4 mm to (-234.9, -995.7), turned to 0 degrees
- moved C65 1053.3 mm to (-195.6, -1002.0), turned to 0 degrees
- moved C60 1052.7 mm to (-210.8, -1002.0), turned to 0 degrees
- moved C61 1050.4 mm to (-205.7, -1002.0), turned to 0 degrees
- moved R23 1048.4 mm to (-151.1, -995.7), turned to 0 degrees
- moved C28 1018.4 mm to (-231.1, -1002.0), turned to 0 degrees
- moved C36 1013.0 mm to (-215.9, -1002.0), turned to 0 degrees
- moved C34 1010.9 mm to (-226.1, -1002.0), turned to 0 degrees
- moved C35 1008.5 mm to (-221.0, -1002.0), turned to 0 degrees
- moved C4 1007.8 mm to (-254.0, -995.7), turned to 0 degrees
- moved C27 1005.9 mm to (-247.7, -995.7), turned to 0 degrees
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Connections:
- removed net 12V_PG: 12V_REG.19, R40.1, U$66.P$1
- removed net 5V_PG: 5V_REG.19, R3.1, U$1.P$1
- removed net N$32: 12V_REG.21, 12V_REG.22, 12V_REG.8, 12V_REG.9, C41.2, L2.P$1
- removed net N$4: 5V_PG.A, R2.1
- removed net N$40: 5V_REG.21, 5V_REG.22, 5V_REG.8, 5V_REG.9, C65.2, L1.P$1
- removed net N$5: R2.2, U$1.P$2
- removed net N$78: LED2.A, R38.1
- removed net N$79: R38.2, U$66.P$2
- new net N$10: R6.P$1, U$41.P$6
- new net N$14: JP1.2, U$25.P$3
- new net N$16: R5.P$1, U$25.P$6
- new net N$19: C4.1, U$48.TMR
- new net N$22: R23.2, R28.1
- new net N$23: R26.2, U$49.1
- new net N$26: R12.1, U$48.SENSE, U$50.TAB
- new net N$29: U$48.DGATE, U$50.1
- new net N$35: R13.2, R17.1, U$51.UV
- new net N$36: R14.1, R20.2, U$51.FB
- new net N$39: R27.1, R9.2, U$48.UV
- new net N$41: R16.1, U$51.HGATE
- new net N$46: R15.1, U$51.SENSE, U$53.TAB
- new net N$50: R23.1, R24.2, U$48.FB
- new net N$51: C60.1, R22.2, U$56.P$2
- new net N$62: JP3.2, U$48.SHDN, U$51.SHDN, U$56.P$4
- new net N$63: LED1.P$1, R37.1
- new net N$64: PMOS1.P$1, R36.1, U$51.FLT
- new net N$65: AUDIO.P$1, R37.2, R39.1
- new net N$66: LED3.P$1, R42.1
- new net N$67: PMOS2.P$1, R41.1, U$48.FLT
- new net N$68: AUDIO1.P$1, R42.2, R43.1
- new net N$69: R44.1, U$55.3
- new net N$70: LED4.C, R44.2
- new net N$75: R46.1, U$58.3
- new net N$76: LED5.P$2, R46.2
- new net N$80: POT.P$2, TEST-PTS.2, U$60.P$2
- new net N$81: LED6.P$1, R48.1, U$60.P$1
- new net N$82: POT1.P$2, TEST-PTS1.2, U$61.P$2
- new net N$83: LED7.P$1, R49.1, U$61.P$1
- new net N$84: R47.1, U$51.ENOUT, U$58.1
- new net N$85: R45.1, U$48.ENOUT, U$55.1
- new net N$86: LED8.P$1, R50.1
- new net N$87: LED9.P$1, R51.1
- new net N$88: PMOS1.P$2, R39.2
- new net N$89: PMOS2.P$2, R43.2
- new net SHDN_SW: 2PIN_5.P$1, R22.1, R29.1, U$62.1, U$62.2
- new net V_BATT: C28.1, C65.1, JP6.P$1, R12.2, R15.2, R19.2, R28.2, U$48.OUT, U$51.OUT, U$54.P$2
- new net V_BATT1: BATT1_IN.P$1, C34.1, C61.1, LED4.A, PMOS2.P$3, POT1.P$1, R27.2, R41.2, R45.2, R49.2, R51.2, U$48.VCC, U$49.TAB, U$57.P$3
- new net V_BATT2: BATT2_IN.P$1, C35.1, LED5.P$1, PMOS1.P$3, POT.P$1, R17.2, R36.2, R47.2, R48.2, R50.2, U$51.VCC, U$52.TAB
- new net V_SHORE: SHORE_IN.P$1
- net +12V: now also U$1.P$2, U$63.P$2, U$64.P$2; no longer TVS1.P$1, TVS2.P$1, TVS3.P$1
- net +5V: now also U$21.1, U$21.2, U$42.1, U$42.2, U$43.1, U$43.2, U$44.1, U$44.2, U$46.1, U$46.2, U$47.1, U$47.2; no longer 5-TVS_1.P$1, 5-TVS_1.P$3, 5-TVS_1.P$4, 5-TVS_1.P$6, 5-TVS_2.P$1, 5-TVS_2.P$3, 5-TVS_2.P$4, 5-TVS_2.P$6, 5-TVS_3.P$1, 5-TVS_3.P$3, 5-TVS_3.P$4, 5-TVS_3.P$6, U$21.P$2
- net 12V_CURR: now also C38.P$1, C40.1, U$41.P$5, U$41.P$7; no longer 12V_REG.1, C28.1, C35.1, C36.P$1, L2.P$2, R15.2
- net 5V: now also C36.1, C62.1, JP3.1, R29.2, U$56.P$5, U$57.P$2, U$57.P$4, U$65.1, U$65.2
- net 5V_CURR: now also C50.P$1, C51.1, U$25.P$5, U$25.P$7; no longer 5V_REG.1, C42.1, C61.1, C62.P$1, L1.P$2, R23.2
- net CPU_ON: no longer 12V_REG.14
- net GND: now also 2PIN_5.P$2, AUDIO.P$2, AUDIO1.P$2, BATT1_IN.P$2, BATT2_IN.P$2, C28.2, C36.2, C38.P$2, C50.P$2, C51.2, C62.2, C65.2, CIN1.2, CIN2.2, CIN3.2, CIN4.2, JP6.P$2, LED1.P$2, LED3.P$2, LED6.P$2, LED7.P$2, LED8.P$2, LED9.P$2, POT.P$3, POT1.P$3, R13.1, R20.1, R5.P$2, R6.P$2, R9.1, SHORE_IN.P$2, TEST-PTS.1, TEST-PTS1.1, U$1.P$1, U$10.3, U$13.3, U$16.3, U$22.3, U$25.P$1, U$25.P$2, U$26.3, U$28.3, U$30.3, U$31.3, U$32.3, U$33.3, U$34.3, U$38.3, U$41.P$1, U$41.P$2, U$42.3, U$43.3, U$44.3, U$46.3, U$47.3, U$48.GND, U$48.OV, U$51.GND, U$51.OV, U$54.P$1, U$55.2, U$56.P$3, U$57.P$1, U$58.2, U$59.3, U$60.P$3, U$61.P$3, U$62.3, U$63.P$1, U$64.P$1, U$65.3; no longer 12V_REG.10, 12V_REG.11, 12V_REG.18, 12V_REG.6, 12V_REG.7, 5-TVS_1.P$2, 5-TVS_1.P$5, 5-TVS_2.P$2, 5-TVS_2.P$5, 5-TVS_3.P$2, 5-TVS_3.P$5, 5V_PG.C, 5V_REG.10, 5V_REG.11, 5V_REG.18, 5V_REG.6, 5V_REG.7, C36.P$2, C38.2, C39.2, C62.P$2, C63.2, JP3.P1,1, JP3.P1,2, JP3.P1,3, JP3.P1,4, JP3.P1,5, JP3.P1,6, JP3.P2,1, JP3.P2,2, JP3.P2,3, JP3.P2,4, JP3.P2,5, JP3.P2,6, LED2.C, R14.1, R16.1, R17.1, TVS1.P$2, TVS2.P$2, TVS3.P$2, U$10.P$1, U$13.P$1, U$16.P$1, U$22.P$1, U$26.P$1, U$28.P$1, U$30.P$1, U$31.P$1, U$32.P$1, U$33.P$1, U$34.P$1, U$38.P$1, U$59.P$1
- net N$1: now also R26.1, U$48.HGATE; no longer 12V_REG.15, R14.2
- net N$42: now also C27.1, U$51.TMR; no longer 5V_REG.20, C42.2, R23.1, R24.2
- net N$43: now also R14.2, R19.1; no longer 5V_REG.3, C65.1
- net N$44: now also U$52.1; no longer 12V_REG.20, C28.2, R15.1
- net N$45: now also U$51.SOURCE, U$52.3, U$53.3; no longer 12V_REG.3, C41.1
- net N$48: now also U$51.DGATE, U$53.1; no longer 5V_REG.2, C63.1
- net N$54: now also U$48.SOURCE, U$49.3, U$50.3; no longer 12V_REG.2, C39.1
- net N$61: now also U$59.1, U$59.2; no longer U$59.P$2
- net N$8: now also JP2.2, U$41.P$3; no longer 5V_REG.15, R17.2
- net N$9: now also U$21.3; no longer U$21.P$1
- net VIN: now also CIN1.1, CIN2.1, CIN3.1, CIN4.1, U$25.P$4, U$41.P$4; no longer 12V_REG.13, 12V_REG.4, 5V_REG.13, 5V_REG.14, 5V_REG.4, C27.1, C34.1, C38.1, C4.1, C40.1, C60.1, JP3.1, JP3.10, JP3.11, JP3.12, JP3.13, JP3.14, JP3.15, JP3.16, JP3.17, JP3.18, JP3.19, JP3.2, JP3.20, JP3.21, JP3.22, JP3.23, JP3.24, JP3.25, JP3.26, JP3.27, JP3.28, JP3.29, JP3.3, JP3.30, JP3.31, JP3.32, JP3.33, JP3.34, JP3.35, JP3.36, JP3.37, JP3.38, JP3.39, JP3.4, JP3.40, JP3.41, JP3.42, JP3.43, JP3.44, JP3.45, JP3.46, JP3.47, JP3.48, JP3.49, JP3.5, JP3.50, JP3.51, JP3.52, JP3.53, JP3.54, JP3.55, JP3.56, JP3.57, JP3.58, JP3.59, JP3.6, JP3.60, JP3.61, JP3.62, JP3.63, JP3.64, JP3.65, JP3.66, JP3.67, JP3.68, JP3.69, JP3.7, JP3.70, JP3.71, JP3.72, JP3.73, JP3.74, JP3.75, JP3.76, JP3.77, JP3.78, JP3.79, JP3.8, JP3.80, JP3.9, R3.2, R40.2, U$1.P$3, U$66.P$3
- net V_THRUST: now also U$32.1, U$32.2, U$33.1, U$33.2, U$34.1, U$34.2, U$38.1, U$38.2; no longer U$32.P$2, U$33.P$2, U$34.P$2, U$38.P$2
- net V_THRUST1: now also U$31.1, U$31.2; no longer U$31.P$2
- net V_THRUST2: now also U$30.1, U$30.2; no longer U$30.P$2
- net V_THRUST3: now also U$26.1, U$26.2; no longer U$26.P$2
- net V_THRUST4: now also U$28.1, U$28.2; no longer U$28.P$2
- net V_THRUST5: now also U$22.1, U$22.2; no longer U$22.P$2
- net V_THRUST6: now also U$13.1, U$13.2; no longer U$13.P$2
- net V_THRUST7: now also U$16.1, U$16.2; no longer U$16.P$2
- net V_THRUST8: now also U$10.1, U$10.2; no longer U$10.P$2
Routing:
- net VIN: track 101.7 -> 0.00 mm, vias 15 -> 1
- net 5V_CURR: track 46.8 -> 0.00 mm
- net 12V_CURR: track 38.9 -> 0.00 mm
- net GND: track 210.0 -> 176.6 mm, vias 66 -> 56
- net 12V_PG: track 32.0 -> 0.00 mm, vias 2 -> 0
- net N$40: track 27.2 -> 0.00 mm
- net N$32: track 26.4 -> 0.00 mm
- net 5V_PG: track 16.8 -> 0.00 mm, vias 2 -> 0
- net N$5: track 14.2 -> 0.00 mm
- net N$44: track 8.91 -> 0.00 mm
- net N$42: track 8.91 -> 0.00 mm
- net N$54: track 5.87 -> 0.00 mm
- net N$48: track 5.87 -> 0.00 mm
- net N$45: track 4.28 -> 0.00 mm
- net V_THRUST: track 456.9 -> 461.0 mm
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
Commit message: 
Parts:
- removed POT, POT1: 10k, resistor:PTV09A-4
- added R2, R3: (no value), resistor:RTRIM3314J
- added U$66: VTVSDO-219AB, diode:DO-219AB
- added U$67, U$68: VTVSSOT323, diode:SOT323-R
- added U$69, U$70, U$71, U$72, U$73, U$74, U$75, U$76: TEST_PT534-5004, resistor:534-5004
- R36, R41: value 20k -> 1MO
Connections:
- net +12V: now also U$70.P$1
- net +5V: now also U$69.P$1
- net GND: now also R2.1, R3.1, U$66.P$1, U$67.3, U$68.3; no longer POT.P$3, POT1.P$3
- net N$80: now also R2.2; no longer POT.P$2
- net N$82: now also R3.2; no longer POT1.P$2
- net SCL_5V: now also U$71.P$1
- net SDA_5V: now also U$72.P$1
- net V_BATT1: now also R3.3, U$68.1, U$68.2, U$75.P$1; no longer POT1.P$1
- net V_BATT2: now also R2.3, U$67.1, U$67.2, U$74.P$1; no longer POT.P$1
- net V_SHORE: now also U$66.P$2, U$73.P$1
- net V_THRUST: now also U$76.P$1

Commit message: 
Parts:
- removed C32: 1u, resistor:C0805
- removed JP_5V: (no value), pinhead:1X02
- removed R1: 10k, resistor:R0805
- removed R18: 510, resistor:R0805
- removed R21: 6.8k, resistor:R0805
- removed SW_CPU: KK254_VERT_2PIN"", molex:KK254_VERT_2PIN
- removed U$59, U$65: VTVSSOT323, diode:SOT323-R
- added 2PIN_2, 2PIN_3: KK254_VERT_2PIN"", molex:KK254_VERT_2PIN
- added JP4, JP5: (no value), pinhead:1X02
- JP6: value 2_SUPERSABRE -> (none); device molex:SUPERSABRE_2CIRCUIT -> pinhead:1X02
- R45, R47: value 20k -> 1MO
- U$3: value TIVA-C_EVAL -> TEST_PT534-5004; device texas:TIVA-C_EVAL -> resistor:534-5004
- U$45: value 74LVC1G14 -> VTVSDO-219AB; device NXP:TSSOP5 -> diode:DO-219AB
- U$54: value VTVSDO-219AB -> TEST_PT534-5004; device diode:DO-219AB -> resistor:534-5004
- moved U$45 1235.1 mm to (-284.5, -1219.2), turned to 0 degrees
- moved U$54 1232.4 mm to (-279.4, 224.8)
- moved JP6 359.6 mm to (-278.1, -1285.2)
- moved U$3 249.9 mm to (-279.4, 241.3)
Connections:
- removed net AIN0: U$3.3-9
- removed net AIN1: U$3.3-8
- removed net AIN10: U$3.1-7
- removed net AIN11: U$3.1-2
- removed net AIN2: U$3.3-7
- removed net AIN3: U$3.2-3
- removed net AIN4: U$3.3-6
- removed net AIN5: U$3.3-5
- removed net AIN8: U$3.1-6
- removed net AIN9: U$3.1-5
- removed net CPU_ON: JP_5V.2, U$45.P$4
- removed net N$59: C32.1, R18.2, U$45.P$2
- removed net N$61: R18.1, R21.1, SW_CPU.P$1, U$59.1, U$59.2
- removed net N$7: C30.1, U$24.6, U$24.7, U$24.8, U$7.AA, U$7.AB
- removed net SCL_5V: 12V_CURR_ADC.P$1, 12V_VOLTAGE.P$5, 5V_CURR_ADC.P$1, 5V_VOLTAGE.P$5, R8.1, THRUSTER_CURR_ADC.14, U$3.1-9, U$71.P$1, U1.26, V-THRUST_CURR_ADC.P$1, V-THRUST_VOLTAGE.P$5
- removed net SDA_5V: 12V_CURR_ADC.P$8, 12V_VOLTAGE.P$6, 5V_CURR_ADC.P$8, 5V_VOLTAGE.P$6, R7.1, THRUSTER_CURR_ADC.15, U$3.1-10, U$72.P$1, U1.27, V-THRUST_CURR_ADC.P$8, V-THRUST_VOLTAGE.P$6
- removed net TIVA_!RST!: R1.1, U$3.2-5
- removed net V_BATT: C28.1, C65.1, JP6.P$1, R12.2, R15.2, R19.2, R28.2, U$48.OUT, U$51.OUT, U$54.P$2
- removed net V_SHORE: SHORE_IN.P$1, U$66.P$2, U$73.P$1
- new net N$4: C30.1, JP4.2, U$24.6, U$24.7, U$24.8, U$45.P$2, U$7.AA, U$7.AB
- new net SCL: 12V_CURR_ADC.P$1, 12V_VOLTAGE.P$5, 5V_CURR_ADC.P$1, 5V_VOLTAGE.P$5, JP5.2, R8.1, THRUSTER_CURR_ADC.14, U$71.P$1, U1.26, V-THRUST_CURR_ADC.P$1, V-THRUST_VOLTAGE.P$5
- new net SDA: 12V_CURR_ADC.P$8, 12V_VOLTAGE.P$6, 5V_CURR_ADC.P$8, 5V_VOLTAGE.P$6, JP5.1, R7.1, THRUSTER_CURR_ADC.15, U$72.P$1, U1.27, V-THRUST_CURR_ADC.P$8, V-THRUST_VOLTAGE.P$6
- net +12V: now also JP4.1
- net +3V3: now also 2PIN_2.P$1, U$3.P$1; no longer U$3.1-1
- net +5V: now also 12V_CURR_ADC.P$5, 2PIN_3.P$1; no longer R1.2, R21.2, U$3.3-1, U$45.P$5
- net 5V: no longer 12V_CURR_ADC.P$5, U$65.1, U$65.2
- net GND: now also 2PIN_2.P$2, 2PIN_3.P$2, JP1.1, JP2.1, U$45.P$1; no longer C32.2, JP6.P$2, SW_CPU.P$2, U$3.2-1, U$3.3-2, U$45.P$3, U$54.P$1, U$59.3, U$65.3
- net SCL-3V3: now also JP6.2; no longer U$3.2-7
- net SDA-3V3: now also JP6.1; no longer U$3.2-6
- net VIN: now also C28.1, C65.1, R12.2, R15.2, R19.2, R28.2, SHORE_IN.P$1, U$48.OUT, U$51.OUT, U$66.P$2, U$73.P$1; no longer JP_5V.1
- net V_THRUST: now also U$54.P$1
Routing:
- net SCL_5V: track 30.2 -> 0.00 mm, vias 3 -> 0
- net SCL: track 0.00 -> 30.2 mm, vias 0 -> 3
- net CPU_ON: track 24.9 -> 0.00 mm, vias 1 -> 0
- net N$61: track 15.2 -> 0.00 mm
- net GND: track 176.6 -> 166.6 mm, vias 56 -> 54
- net SDA_5V: track 8.36 -> 0.00 mm, vias 1 -> 0
- net SDA: track 0.00 -> 8.36 mm, vias 0 -> 1
- net N$59: track 5.69 -> 0.00 mm
- net 5V: track 2.92 -> 0.00 mm
- net +5V: track 72.4 -> 71.2 mm
Other:
- board text added: "Designed By: Ben Hurwitz and Alex Jiao Robotics at Maryland, 2017"
- board text removed: "Designed By: Ben Hurwitz Robotics at Maryland, 2017"
