File: Project QUBO/eagleDesigns/Jr Support/Jr Support/jr-support_v4.sch (EAGLE design)
At the start: 207 parts, among them U1 PCA9685

Commit message: updated jr support
Parts:
- removed 12V_REG, 5V_REG: LT8640, linear:LT8640
- removed 5-TVS_1, 5-TVS_2, 5-TVS_3: BZA408B, diodes:BZA408B
- removed 5V_PG: Red, led:LEDCHIP-LED0805
- removed C39, C63: 1u, resistor:C-USC0805
- removed C41: 0.1u, resistor:C-USC0805
- removed C42: 15p, resistor:C-USC0805
- removed L1, L2: 2.2u, resistor:L-USL0740
- removed LED2: RED, led:LEDCHIP-LED0805
- removed R2, R38: 1.2k, resistor:R-US_R0805
- removed R3, R40: 50k, resistor:R-US_R0805
- removed TVS1, TVS2, TVS3: (no value), diode:ESD12VD3B
- removed U$66: SSM3J353F, transistors:SSM3J353F
- added 2PIN_5, AUDIO, AUDIO1, BATT1_IN, BATT2_IN, SHORE_IN: KK254_VERT_2PIN"", molex:KK254_VERT_2PIN""
- added C50: 330 uF, resistor:CPOL-USCKR_D10
- added C51: .1 uF, resistor:C-USC0805
- added CIN1, CIN2, CIN3, CIN4: 2.2 uF, resistor:C-USC1210
- added JP1, JP2: (no value), jumper:JP1E
- added JP6: 2_SUPERSABRE, molex:2_SUPERSABRE
- added LED1, LED3: Red, led:0805_LED
- added LED4: Green, led:LEDCHIPLED_0805
- added LED5, LED8, LED9: Green, led:0805_LED
- added LED6, LED7: Yellow, led:0805_LED
- added PMOS1, PMOS2: SSM3J353F, transistors:SSM3J353F
- added POT, POT1: 10k, resistor:R-TRIMMPTV09A-4
- added R12: 5m, resistor:R-US_R0805
- added R13: 20.8k, resistor:R-US_R0805
- added R19, R28: 8.2k, resistor:R-US_R0805
- added R20: 5.1k, resistor:R-US_R0805
- added R22: 510, resistor:R-US_R0805
- added R26: 10\, resistor:R-US_R0805
- added R27: 200k, resistor:R-US_R0805
- added R29: 6.8k, resistor:R-US_R0805
- added R36, R41, R45, R47: 20k, resistor:R-US_R0805
- added R37, R42: 430, resistor:R-US_R0805
- added R39, R43, R48, R49: 330, resistor:R-US_R0805
- added R44, R46: 1.2k, resistor:R-US_R0805
- added R5: 21kO, resistor:R-US_RC55/H8
- added R50, R51: 1.5k, resistor:R-US_R0805
- added R6: 2.61kO, resistor:R-US_RC55/H8
- added R9: 12k, resistor:R-US_R0805
- added TEST-PTS, TEST-PTS1: 0, resistor:R-US_V526-0
- added U$25, U$41: PTN78060W, texas:PTN78060W
- added U$42, U$43, U$44, U$46, U$47, U$62, U$65: VTVSSOT323, diode:VTVSSOT323
- added U$48, U$51: LTC4364MSOP, linear:LTC4364MSOP
- added U$49, U$50, U$52, U$53: STD95N2LH5, transistors:STD95N2LH5
- added U$54, U$63, U$64: VTVSDO-219AB, diode:VTVSDO-219AB
- added U$55, U$58: BSS138CT-NDSOT23, transistor-fet:BSS138CT-NDSOT23
- added U$56: 74LVC1G14, NXP:74LVC1G14
- added U$57: NCP1117, ONSemi:NCP1117
- added U$60, U$61: TL431DBZ, texas:TL431DBZ
- 12V_OUT, 5V_OUT, V-THRUST_OUT: device molex:KK254_VERT_2PIN22-29-2021 -> molex:KK254_VERT_2PIN""
- 2PIN_1, CAMERA1, CAMERA2, ETHERNET, FAN1, FAN2, SW_CPU: value KK254_VERT_2PIN22-29-2021 -> KK254_VERT_2PIN""; device molex:KK254_VERT_2PIN22-29-2021 -> molex:KK254_VERT_2PIN""
- C27: value 10u -> 0.22u
- C28: value 15p -> 22u
- C35: value 22u -> 1u
- C36: value 220u -> 1u; device resistor:CPOL-USC-F80 -> resistor:C-USC0805
- C38: value 1u -> 330 uF; device resistor:C-USC0805 -> resistor:CPOL-USCKR_D10
- C4: value 1u -> 0.22u
- C40: value 10u -> .1 uF
- C61: value 22u -> 10u
- C62: value 220u -> 10u; device resistor:CPOL-USC-F80 -> resistor:C-USC0805
- C65: value 0.1u -> 22u
- JP3: value MPTC-01-80 -> (none); device samtec:MPTC-01-80 -> pinhead:PINHD-1X2
- R14: value 41.2k -> 51k
- R15: value 1M -> 5m
- R16: value 88.7k -> 10\
- R17: value 41.2k -> 200k
- R23: value 1M -> 51k
- R24: value 243k -> 5.1k
- U$1: value SSM3J353F -> VTVSDO-219AB; device transistors:SSM3J353F -> diode:VTVSDO-219AB
- U$10, U$13, U$16, U$21, U$22, U$26, U$28, U$30, U$31, U$32, U$33, U$34, U$38, U$59: value VTVS -> VTVSSOT323; device diode:VTVS -> diode:VTVSSOT323
Connections:
- removed net 12V_PG: 12V_REG.PG, R40.1, U$66.G
- removed net 5V_PG: 5V_REG.PG, R3.1, U$1.G
- removed net N$32: 12V_REG.SW, C41.2, L2.1
- removed net N$4: 5V_PG.A, R2.1
- removed net N$40: 5V_REG.SW, C65.2, L1.1
- removed net N$5: R2.2, U$1.D
- removed net N$78: LED2.A, R38.1
- removed net N$79: R38.2, U$66.D
- new net N$10: R6.1, U$41.VOADJUST
- new net N$14: JP1.2, U$25.!INHIBIT!
- new net N$16: R5.1, U$25.VOADJUST
- new net N$19: C4.1, U$48.TMR
- new net N$22: R23.2, R28.1
- new net N$23: R26.2, U$49.G
- new net N$26: R12.1, U$48.SENSE, U$50.D
- new net N$29: U$48.DGATE, U$50.G
- new net N$35: R13.2, R17.1, U$51.UV
- new net N$36: R14.1, R20.2, U$51.FB
- new net N$39: R27.1, R9.2, U$48.UV
- new net N$41: R16.1, U$51.HGATE
- new net N$46: R15.1, U$51.SENSE, U$53.D
- new net N$50: R23.1, R24.2, U$48.FB
- new net N$51: C60.1, R22.2, U$56.IN
- new net N$62: JP3.2, U$48.!SHDN!, U$51.!SHDN!, U$56.OUT
- new net N$63: LED1.A, R37.1
- new net N$64: PMOS1.G, R36.1, U$51.!FAULT!
- new net N$65: AUDIO.P$1, R37.2, R39.1
- new net N$66: LED3.A, R42.1
- new net N$67: PMOS2.G, R41.1, U$48.!FAULT!
- new net N$68: AUDIO1.P$1, R42.2, R43.1
- new net N$69: R44.1, U$55.D
- new net N$70: LED4.C, R44.2
- new net N$75: R46.1, U$58.D
- new net N$76: LED5.C, R46.2
- new net N$80: POT.S, TEST-PTS.2, U$60.REF
- new net N$81: LED6.A, R48.1, U$60.C
- new net N$82: POT1.S, TEST-PTS1.2, U$61.REF
- new net N$83: LED7.A, R49.1, U$61.C
- new net N$84: R47.1, U$51.ENOUT, U$58.G
- new net N$85: R45.1, U$48.ENOUT, U$55.G
- new net N$86: LED8.A, R50.1
- new net N$87: LED9.A, R51.1
- new net N$88: PMOS1.D, R39.2
- new net N$89: PMOS2.D, R43.2
- new net SHDN_SW: 2PIN_5.P$1, R22.1, R29.1, U$62.C
- new net V_BATT: C28.1, C65.1, JP6.P$1, R12.2, R15.2, R19.2, R28.2, U$48.OUT, U$51.OUT, U$54.C
- new net V_BATT1: BATT1_IN.P$1, C34.1, C61.1, LED4.A, PMOS2.S, POT1.A, R27.2, R41.2, R45.2, R49.2, R51.2, U$48.VCC, U$49.D, U$57.VIN
- new net V_BATT2: BATT2_IN.P$1, C35.1, LED5.A, PMOS1.S, POT.A, R17.2, R36.2, R47.2, R48.2, R50.2, U$51.VCC, U$52.D
- new net V_SHORE: SHORE_IN.P$1
- net +12V: now also U$1.C, U$63.C, U$64.C; no longer TVS1.P$1, TVS2.P$1, TVS3.P$1
- net +5V: now also U$42.C, U$43.C, U$44.C, U$46.C, U$47.C; no longer 5-TVS_1.P$1, 5-TVS_1.P$3, 5-TVS_1.P$4, 5-TVS_1.P$6, 5-TVS_2.P$1, 5-TVS_2.P$3, 5-TVS_2.P$4, 5-TVS_2.P$6, 5-TVS_3.P$1, 5-TVS_3.P$3, 5-TVS_3.P$4, 5-TVS_3.P$6
- net 12V_CURR: now also C38.+, C40.1, U$41.VO, U$41.VOSENSE; no longer 12V_REG.BIAS, C28.1, C35.1, C36.+, L2.2, R15.2
- net 5V: now also C36.1, C62.1, JP3.1, R29.2, U$56.VDD, U$57.VOUT, U$65.C
- net 5V_CURR: now also C50.+, C51.1, U$25.VO, U$25.VOSENSE; no longer 5V_REG.BIAS, C42.1, C61.1, C62.+, L1.2, R23.2
- net CPU_ON: no longer 12V_REG.EN/UV
- net GND: now also 2PIN_5.P$2, AUDIO.P$2, AUDIO1.P$2, BATT1_IN.P$2, BATT2_IN.P$2, C28.2, C36.2, C38.-, C50.-, C51.2, C62.2, C65.2, CIN1.2, CIN2.2, CIN3.2, CIN4.2, JP6.P$2, LED1.C, LED3.C, LED6.C, LED7.C, LED8.C, LED9.C, POT.E, POT1.E, R13.1, R20.1, R5.2, R6.2, R9.1, SHORE_IN.P$2, TEST-PTS.1, TEST-PTS1.1, U$1.A, U$25.GND1, U$25.GND2, U$41.GND1, U$41.GND2, U$42.A, U$43.A, U$44.A, U$46.A, U$47.A, U$48.GND, U$48.OV, U$51.GND, U$51.OV, U$54.A, U$55.S, U$56.GND, U$57.GND, U$58.S, U$60.A, U$61.A, U$62.A, U$63.A, U$64.A, U$65.A; no longer 12V_REG.GND, 12V_REG.GND-1, 12V_REG.GND-2, 5-TVS_1.P$2, 5-TVS_1.P$5, 5-TVS_2.P$2, 5-TVS_2.P$5, 5-TVS_3.P$2, 5-TVS_3.P$5, 5V_PG.C, 5V_REG.GND, 5V_REG.GND-1, 5V_REG.GND-2, C36.-, C38.2, C39.2, C62.-, C63.2, JP3.POWER1, JP3.POWER2, LED2.C, R14.1, R16.1, R17.1, TVS1.P$2, TVS2.P$2, TVS3.P$2
- net N$1: now also R26.1, U$48.HGATE; no longer 12V_REG.RT, R14.2
- net N$42: now also C27.1, U$51.TMR; no longer 5V_REG.FB, C42.2, R23.1, R24.2
- net N$43: now also R14.2, R19.1; no longer 5V_REG.BST, C65.1
- net N$44: now also U$52.G; no longer 12V_REG.FB, C28.2, R15.1
- net N$45: now also U$51.SOURCE, U$52.S, U$53.S; no longer 12V_REG.BST, C41.1
- net N$48: now also U$51.DGATE, U$53.G; no longer 5V_REG.INTV-CC, C63.1
- net N$54: now also U$48.SOURCE, U$49.S, U$50.S; no longer 12V_REG.INTV-CC, C39.1
- net N$8: now also JP2.2, U$41.!INHIBIT!; no longer 5V_REG.RT, R17.2
- net VIN: now also CIN1.1, CIN2.1, CIN3.1, CIN4.1, U$25.VI, U$41.VI; no longer 12V_REG.VIN-1, 12V_REG.VIN-2, 5V_REG.EN/UV, 5V_REG.VIN-1, 5V_REG.VIN-2, C27.1, C34.1, C38.1, C4.1, C40.1, C60.1, JP3.P$1, JP3.P$10, JP3.P$11, JP3.P$12, JP3.P$13, JP3.P$14, JP3.P$15, JP3.P$16, JP3.P$17, JP3.P$18, JP3.P$19, JP3.P$2, JP3.P$20, JP3.P$21, JP3.P$22, JP3.P$23, JP3.P$24, JP3.P$25, JP3.P$26, JP3.P$27, JP3.P$28, JP3.P$29, JP3.P$3, JP3.P$30, JP3.P$31, JP3.P$32, JP3.P$33, JP3.P$34, JP3.P$35, JP3.P$36, JP3.P$37, JP3.P$38, JP3.P$39, JP3.P$4, JP3.P$40, JP3.P$41, JP3.P$42, JP3.P$43, JP3.P$44, JP3.P$45, JP3.P$46, JP3.P$47, JP3.P$48, JP3.P$49, JP3.P$5, JP3.P$50, JP3.P$51, JP3.P$52, JP3.P$53, JP3.P$54, JP3.P$55, JP3.P$56, JP3.P$57, JP3.P$58, JP3.P$59, JP3.P$6, JP3.P$60, JP3.P$61, JP3.P$62, JP3.P$63, JP3.P$64, JP3.P$65, JP3.P$66, JP3.P$67, JP3.P$68, JP3.P$69, JP3.P$7, JP3.P$70, JP3.P$71, JP3.P$72, JP3.P$73, JP3.P$74, JP3.P$75, JP3.P$76, JP3.P$77, JP3.P$78, JP3.P$79, JP3.P$8, JP3.P$80, JP3.P$9, R3.2, R40.2, U$1.S, U$66.S
Other:
- note added: "The blue LED will turn on when the battery voltage drops below a level given by: (2.5V)(10kO) ----------------- POT where POT is the resistance of the potentiometer."
- note removed: "5V TVS"
- note removed: "PG is an open-drain fault pin."
- moved on the sheet: C27, C28, C34, C35, C4, C40, C60, C61, C65, R14, R15, R16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

Commit message: 
Parts:
- removed POT, POT1: 10k, resistor:R-TRIMMPTV09A-4
- added R2, R3: (no value), resistor:R-TRIMM3314J
- added U$66: VTVSDO-219AB, diode:VTVSDO-219AB
- added U$67, U$68: VTVSSOT323, diode:VTVSSOT323
- added U$69, U$70, U$71, U$72, U$73, U$74, U$75, U$76: TEST_PT534-5004, resistor:TEST_PT534-5004
- R36, R41: value 20k -> 1MO
Connections:
- net +12V: now also U$70.1
- net +5V: now also U$69.1
- net GND: now also R2.E, R3.E, U$66.A, U$67.A, U$68.A; no longer POT.E, POT1.E
- net N$80: now also R2.S; no longer POT.S
- net N$82: now also R3.S; no longer POT1.S
- net SCL_5V: now also U$71.1
- net SDA_5V: now also U$72.1
- net V_BATT1: now also R3.A, U$68.C, U$75.1; no longer POT1.A
- net V_BATT2: now also R2.A, U$67.C, U$74.1; no longer POT.A
- net V_SHORE: now also U$66.C, U$73.1
- net V_THRUST: now also U$76.1

Commit message: 
Parts:
- removed C32: 1u, resistor:C-USC0805
- removed JP_5V: (no value), pinhead:PINHD-1X2
- removed R1: 10k, resistor:R-US_R0805
- removed R18: 510, resistor:R-US_R0805
- removed R21: 6.8k, resistor:R-US_R0805
- removed SW_CPU: KK254_VERT_2PIN"", molex:KK254_VERT_2PIN""
- removed U$59, U$65: VTVSSOT323, diode:VTVSSOT323
- added 2PIN_2, 2PIN_3: KK254_VERT_2PIN"", molex:KK254_VERT_2PIN""
- added JP4, JP5: (no value), pinhead:PINHD-1X2
- JP6: value 2_SUPERSABRE -> (none); device molex:2_SUPERSABRE -> pinhead:PINHD-1X2
- R45, R47: value 20k -> 1MO
- U$3: value TIVA-C_EVAL -> TEST_PT534-5004; device texas:TIVA-C_EVAL -> resistor:TEST_PT534-5004
- U$45: value 74LVC1G14 -> VTVSDO-219AB; device NXP:74LVC1G14 -> diode:VTVSDO-219AB
- U$54: value VTVSDO-219AB -> TEST_PT534-5004; device diode:VTVSDO-219AB -> resistor:TEST_PT534-5004
Connections:
- removed net AIN0: U$3.PE3
- removed net AIN1: U$3.PE2
- removed net AIN10: U$3.PB4
- removed net AIN11: U$3.PB5
- removed net AIN2: U$3.PE1
- removed net AIN3: U$3.PE0
- removed net AIN4: U$3.PD3
- removed net AIN5: U$3.PD2
- removed net AIN8: U$3.PE5
- removed net AIN9: U$3.PE4
- removed net CPU_ON: JP_5V.2, U$45.OUT
- removed net N$59: C32.1, R18.2, U$45.IN
- removed net N$61: R18.1, R21.1, SW_CPU.P$1, U$59.C
- removed net N$7: C30.1, U$24.OUT, U$7.A
- removed net SCL_5V: 12V_CURR_ADC.SCL, 12V_VOLTAGE.SCL, 5V_CURR_ADC.SCL, 5V_VOLTAGE.SCL, R8.1, THRUSTER_CURR_ADC.SCL, U$3.PA6, U$71.1, U1.SCL, V-THRUST_CURR_ADC.SCL, V-THRUST_VOLTAGE.SCL
- removed net SDA_5V: 12V_CURR_ADC.SDA, 12V_VOLTAGE.SDA, 5V_CURR_ADC.SDA, 5V_VOLTAGE.SDA, R7.1, THRUSTER_CURR_ADC.SDA, U$3.PA7, U$72.1, U1.SDA, V-THRUST_CURR_ADC.SDA, V-THRUST_VOLTAGE.SDA
- removed net TIVA_!RST!: R1.1, U$3.!RESET!
- removed net V_BATT: C28.1, C65.1, JP6.P$1, R12.2, R15.2, R19.2, R28.2, U$48.OUT, U$51.OUT, U$54.C
- removed net V_SHORE: SHORE_IN.P$1, U$66.C, U$73.1
- new net N$4: C30.1, JP4.2, U$24.OUT, U$45.C, U$7.A
- new net SCL: 12V_CURR_ADC.SCL, 12V_VOLTAGE.SCL, 5V_CURR_ADC.SCL, 5V_VOLTAGE.SCL, JP5.2, R8.1, THRUSTER_CURR_ADC.SCL, U$71.1, U1.SCL, V-THRUST_CURR_ADC.SCL, V-THRUST_VOLTAGE.SCL
- new net SDA: 12V_CURR_ADC.SDA, 12V_VOLTAGE.SDA, 5V_CURR_ADC.SDA, 5V_VOLTAGE.SDA, JP5.1, R7.1, THRUSTER_CURR_ADC.SDA, U$72.1, U1.SDA, V-THRUST_CURR_ADC.SDA, V-THRUST_VOLTAGE.SDA
- net +12V: now also JP4.1
- net +3V3: now also 2PIN_2.P$1, U$3.1; no longer U$3.3V3
- net +5V: now also 12V_CURR_ADC.VDD, 2PIN_3.P$1; no longer R1.2, R21.2, U$3.5V, U$45.VDD
- net 5V: no longer 12V_CURR_ADC.VDD, U$65.C
- net GND: now also 2PIN_2.P$2, 2PIN_3.P$2, JP1.1, JP2.1, U$45.A; no longer C32.2, JP6.P$2, SW_CPU.P$2, U$3.GND@2-1, U$3.GND@3-2, U$45.GND, U$54.A, U$59.A, U$65.A
- net SCL-3V3: now also JP6.2; no longer U$3.PD0
- net SDA-3V3: now also JP6.1; no longer U$3.PD1
- net VIN: now also C28.1, C65.1, R12.2, R15.2, R19.2, R28.2, SHORE_IN.P$1, U$48.OUT, U$51.OUT, U$66.C, U$73.1; no longer JP_5V.1
- net V_THRUST: now also U$54.1
Other:
- note added: "Embedded System Headers"
- note removed: "NOTE (from the datasheet): The TIVA-C has 5V-tolerant non-driving GPIOs which allows us to have a 5V I2C bus and a 3.3V I2C bus. HOWEVER, pins PD4, PD5, PB0, and PB1 are 3.6V-limited."
- note removed: "Tiva-C"
- moved on the sheet: C33, R10, R11, U$62
