File: Project QUBO/eagleDesigns/BatteryHullBoard/BatteryHullBoard.sch (EAGLE design)
At the start: 7 parts, among them U1 KSK-1E66, U2 CMXSIPSSR

Commit message: 
Parts:
- added R3: 10000, resistor:R-US_R0805
Connections:
- removed net N$6: LED1.C, U2.3
- new net N$4: LED1.C, R3.2
- net GND: now also R3.1
- net N$3: now also U2.3
Other:
- moved on the sheet: LED1
Changed lines of the file:
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@@
 <part name="R2" library="resistor" deviceset="R-US_" device="R0805" value="7700"/>
 <part name="FRAME1" library="frames" deviceset="A5L-LOC" device=""/>
+<part name="R3" library="resistor" deviceset="R-US_" device="R0805" value="10000"/>
 </parts>
 <sheets>
@@
 <instance part="BATTERY" gate="G$1" x="48.26" y="88.9" rot="MR0"/>
 <instance part="ROBOT" gate="G$1" x="124.46" y="78.74"/>
-<instance part="LED1" gate="G$1" x="99.06" y="78.74" rot="R90"/>
+<instance part="LED1" gate="G$1" x="99.06" y="76.2"/>
 <instance part="R1" gate="G$1" x="81.28" y="83.82" rot="R90"/>
 <instance part="R2" gate="G$1" x="81.28" y="71.12" rot="R90"/>
 <instance part="FRAME1" gate="G$1" x="0" y="0"/>
+<instance part="R3" gate="G$1" x="99.06" y="63.5" rot="R90"/>
 </instances>
 <busses>
@@
 <wire x1="81.28" y1="66.04" x2="55.88" y2="66.04" width="0.1524" layer="91"/>
 <wire x1="55.88" y1="66.04" x2="55.88" y2="86.36" width="0.1524" layer="91"/>
+<wire x1="81.28" y1="66.04" x2="81.28" y2="53.34" width="0.1524" layer="91"/>
+<wire x1="81.28" y1="53.34" x2="99.06" y2="53.34" width="0.1524" layer="91"/>
+<junction x="81.28" y="66.04"/>
 <pinref part="ROBOT" gate="G$1" pin="P$2"/>
-<wire x1="116.84" y1="76.2" x2="116.84" y2="66.04" width="0.1524" layer="91"/>
-<wire x1="116.84" y1="66.04" x2="81.28" y2="66.04" width="0.1524" layer="91"/>
-<junction x="81.28" y="66.04"/>
+<wire x1="99.06" y1="53.34" x2="116.84" y2="53.34" width="0.1524" layer="91"/>
+<wire x1="116.84" y1="76.2" x2="116.84" y2="53.34" width="0.1524" layer="91"/>
+<pinref part="R3" gate="G$1" pin="1"/>
+<wire x1="99.06" y1="58.42" x2="99.06" y2="53.34" width="0.1524" layer="91"/>
+<junction x="99.06" y="53.34"/>
+<label x="99.06" y="50.8" size="1.778" layer="95"/>
 </segment>
 <segment>
@@
 <wire x1="81.28" y1="76.2" x2="81.28" y2="78.74" width="0.1524" layer="91"/>
 <pinref part="LED1" gate="G$1" pin="A"/>
-<wire x1="81.28" y1="78.74" x2="96.52" y2="78.74" width="0.1524" layer="91"/>
+<wire x1="81.28" y1="78.74" x2="99.06" y2="78.74" width="0.1524" layer="91"/>
 <junction x="81.28" y="78.74"/>
+<wire x1="114.3" y1="78.74" x2="114.3" y2="88.9" width="0.1524" layer="91"/>
+<pinref part="U2" gate="G$1" pin="3"/>
+<wire x1="114.3" y1="88.9" x2="116.84" y2="88.9" width="0.1524" layer="91"/>
+<wire x1="116.84" y1="88.9" x2="116.84" y2="93.98" width="0.1524" layer="91"/>
+<wire x1="99.06" y1="78.74" x2="114.3" y2="78.74" width="0.1524" layer="91"/>
+<junction x="99.06" y="78.74"/>
 </segment>
 </net>
@@
 </segment>
 </net>
-<net name="N$6" class="0">
-<segment>
-<pinref part="LED1" gate="G$1" pin="C"/>
-<wire x1="104.14" y1="78.74" x2="114.3" y2="78.74" width="0.1524" layer="91"/>
-<wire x1="114.3" y1="78.74" x2="114.3" y2="88.9" width="0.1524" layer="91"/>
-<pinref part="U2" gate="G$1" pin="3"/>
-<wire x1="114.3" y1="88.9" x2="116.84" y2="88.9" width="0.1524" layer="91"/>
-<wire x1="116.84" y1="88.9" x2="116.84" y2="93.98" width="0.1524" layer="91"/>
-</segment>
-</net>
 <net name="N$1" class="0">
 <segment>
@@
 </segment>
 </net>
+<net name="N$4" class="0">
+<segment>
+<pinref part="LED1" gate="G$1" pin="C"/>
+<pinref part="R3" gate="G$1" pin="2"/>
+<wire x1="99.06" y1="71.12" x2="99.06" y2="68.58" width="0.1524" layer="91"/>
+</segment>
+</net>
