File: Project QUBO/eagleDesigns/HypertronicsBoard/Hypertronicsboard.sch (EAGLE design)
At the start: 4 parts

Commit message: Hypertonics board building
I built a lot of the hypertonics board
Parts:
- removed FUSE1, FUSE2, FUSE3, FUSE4: 4A, littelfuse:BOWED-1.25"-FUSECLIPS
- added ADRESS0, ADRESS1, ADRESS2, ADRESS3, ADRESS4, ADRESS5: PULLUP_PULLDOWN0805, resistor:PULLUP_PULLDOWN0805
- added JP1: PWR, molex:2_SUPERSABRE
- added LIL_PWR: 22-23-2021, con-molex_MOD:22-23-2021
- added PWM: PCA9685, NXP:PCA9685
- added U$1, U$2, U$3, U$4: BCS-106-L-D-PE-BE, samtec:BCS-106-L-D-PE-BE
- added U$10, U$11, U$12, U$5, U$6, U$7, U$8, U$9: CONN-RECEPT-2MM-VERT-AU-10POS, samtec:CONN-RECEPT-2MM-VERT-AU-10POS
Connections:
- new net A0: ADRESS0.MID, PWM.A0
- new net A1: ADRESS1.MID, PWM.A1
- new net A2: ADRESS2.MID, PWM.A2
- new net A3: ADRESS3.MID, PWM.A3
- new net A4: ADRESS4.MID, PWM.A4
- new net A5: ADRESS5.MID, PWM.A5
- new net CH0: PWM.CH0, U$10.8
- new net CH1: PWM.CH1, U$10.1
- new net CH2: PWM.CH2, U$10.2
- new net CH3: PWM.CH3, U$10.3
- new net CH4: PWM.CH4, U$10.4
- new net CH5: PWM.CH5, U$10.5
- new net CH6: PWM.CH6, U$10.6
- new net CH7: PWM.CH7, U$10.7
- new net GND: ADRESS0.GND, ADRESS1.GND, ADRESS2.GND, ADRESS3.GND, ADRESS4.GND, ADRESS5.GND, JP1.P$2, LIL_PWR-2.S, PWM.VSS, U$1.2, U$1.3, U$2.2, U$2.3, U$3.1, U$3.4, U$4.1, U$4.4
- new net N$10: U$10.10
- new net N$9: U$10.9
- new net SCL: PWM.SCL, U$5.2
- new net SDA: PWM.SDA, U$5.1
- new net VIN: JP1.P$1, U$1.1, U$1.4, U$2.1, U$2.4, U$3.2, U$3.3, U$4.2, U$4.3
- new net VIN2: ADRESS0.PWR, ADRESS1.PWR, ADRESS2.PWR, ADRESS3.PWR, ADRESS4.PWR, ADRESS5.PWR, LIL_PWR-1.S, PWM.VDD

Commit message: I added a maybe useful cam voltage source
Parts:
- added CAM_PWR1: 22-23-2021, con-molex_MOD:22-23-2021
Connections:
- new net N$1: PWM.!OE
- new net VINCAM: CAM_PWR1-1.S, U$5.10
- net GND: now also CAM_PWR1-2.S, PWM.EXTCLK, U$5.9
Changed lines of the file:
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@@
 <part name="ADRESS4" library="resistor" deviceset="PULLUP_PULLDOWN" device="0805"/>
 <part name="ADRESS5" library="resistor" deviceset="PULLUP_PULLDOWN" device="0805"/>
+<part name="CAM_PWR1" library="con-molex_MOD" deviceset="22-23-2021" device=""/>
 </parts>
 <sheets>
@@
 <attribute name="NAME" x="-37.0586" y="44.45" size="1.778" layer="95" rot="R90"/>
 </instance>
+<instance part="CAM_PWR1" gate="-1" x="-2.54" y="66.04"/>
+<instance part="CAM_PWR1" gate="-2" x="-2.54" y="63.5"/>
 </instances>
 <busses>
@@
 <label x="-73.66" y="58.42" size="1.778" layer="95"/>
 </segment>
+<segment>
+<pinref part="PWM" gate="G$1" pin="EXTCLK"/>
+<wire x1="81.28" y1="66.04" x2="88.9" y2="66.04" width="0.1524" layer="91"/>
+<label x="83.82" y="66.04" size="1.778" layer="95"/>
+</segment>
+<segment>
+<pinref part="CAM_PWR1" gate="-2" pin="S"/>
+<wire x1="-5.08" y1="63.5" x2="-10.16" y2="63.5" width="0.1524" layer="91"/>
+<label x="-10.16" y="63.5" size="1.778" layer="95"/>
+</segment>
+<segment>
+<pinref part="U$5" gate="G$1" pin="9"/>
+<wire x1="-58.42" y1="22.86" x2="-58.42" y2="30.48" width="0.1524" layer="91"/>
+<label x="-58.42" y="30.48" size="1.778" layer="95"/>
+</segment>
 </net>
 <net name="CH1" class="0">
@@
 <pinref part="PWM" gate="G$1" pin="VDD"/>
 <wire x1="81.28" y1="73.66" x2="86.36" y2="73.66" width="0.1524" layer="91"/>
-<label x="81.28" y="73.66" size="1.778" layer="95"/>
+<label x="83.82" y="73.66" size="1.778" layer="95"/>
 </segment>
 <segment>
@@
 </segment>
 </net>
+<net name="VINCAM" class="0">
+<segment>
+<pinref part="CAM_PWR1" gate="-1" pin="S"/>
+<wire x1="-5.08" y1="66.04" x2="-10.16" y2="66.04" width="0.1524" layer="91"/>
+<label x="-10.16" y="66.04" size="1.778" layer="95"/>
+</segment>
+<segment>
+<pinref part="U$5" gate="G$1" pin="10"/>
+<wire x1="-63.5" y1="22.86" x2="-63.5" y2="30.48" width="0.1524" layer="91"/>
+<label x="-71.12" y="30.48" size="1.778" layer="95"/>
+</segment>
+</net>
+<net name="N$1" class="0">
+<segment>
+<pinref part="PWM" gate="G$1" pin="!OE"/>
+<wire x1="81.28" y1="60.96" x2="88.9" y2="60.96" width="0.1524" layer="91"/>
+</segment>
+</net>

Commit message: Nevermind, no camera voltage source
Parts:
- removed CAM_PWR1: 22-23-2021, con-molex_MOD:22-23-2021
Connections:
- removed net VINCAM: CAM_PWR1-1.S, U$5.10
- net GND: no longer CAM_PWR1-2.S, U$5.9
Changed lines of the file:
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@@
 <part name="ADRESS4" library="resistor" deviceset="PULLUP_PULLDOWN" device="0805"/>
 <part name="ADRESS5" library="resistor" deviceset="PULLUP_PULLDOWN" device="0805"/>
-<part name="CAM_PWR1" library="con-molex_MOD" deviceset="22-23-2021" device=""/>
 </parts>
 <sheets>
@@
 <attribute name="NAME" x="-37.0586" y="44.45" size="1.778" layer="95" rot="R90"/>
 </instance>
-<instance part="CAM_PWR1" gate="-1" x="-2.54" y="66.04"/>
-<instance part="CAM_PWR1" gate="-2" x="-2.54" y="63.5"/>
 </instances>
 <busses>
@@
 <label x="83.82" y="66.04" size="1.778" layer="95"/>
 </segment>
-<segment>
-<pinref part="CAM_PWR1" gate="-2" pin="S"/>
-<wire x1="-5.08" y1="63.5" x2="-10.16" y2="63.5" width="0.1524" layer="91"/>
-<label x="-10.16" y="63.5" size="1.778" layer="95"/>
-</segment>
-<segment>
-<pinref part="U$5" gate="G$1" pin="9"/>
-<wire x1="-58.42" y1="22.86" x2="-58.42" y2="30.48" width="0.1524" layer="91"/>
-<label x="-58.42" y="30.48" size="1.778" layer="95"/>
-</segment>
 </net>
 <net name="CH1" class="0">
@@
 </segment>
 </net>
-<net name="VINCAM" class="0">
-<segment>
-<pinref part="CAM_PWR1" gate="-1" pin="S"/>
-<wire x1="-5.08" y1="66.04" x2="-10.16" y2="66.04" width="0.1524" layer="91"/>
-<label x="-10.16" y="66.04" size="1.778" layer="95"/>
-</segment>
-<segment>
-<pinref part="U$5" gate="G$1" pin="10"/>
-<wire x1="-63.5" y1="22.86" x2="-63.5" y2="30.48" width="0.1524" layer="91"/>
-<label x="-71.12" y="30.48" size="1.778" layer="95"/>
-</segment>
-</net>

Commit message: I did a cam
I did a cam on the hypertonics board
Parts:
- removed U$11, U$12, U$8, U$9: CONN-RECEPT-2MM-VERT-AU-10POS, samtec:CONN-RECEPT-2MM-VERT-AU-10POS
Connections:
- net GND: now also U$3.2, U$3.3, U$4.2, U$4.3; no longer U$1.2, U$1.3, U$2.2, U$2.3
- net VIN: now also U$1.2, U$1.3, U$2.2, U$2.3; no longer U$3.2, U$3.3, U$4.2, U$4.3
Changed lines of the file:
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@@
 <part name="U$6" library="samtec" deviceset="CONN-RECEPT-2MM-VERT-AU-10POS" device=""/>
 <part name="U$7" library="samtec" deviceset="CONN-RECEPT-2MM-VERT-AU-10POS" device=""/>
-<part name="U$8" library="samtec" deviceset="CONN-RECEPT-2MM-VERT-AU-10POS" device=""/>
-<part name="U$9" library="samtec" deviceset="CONN-RECEPT-2MM-VERT-AU-10POS" device=""/>
 <part name="U$10" library="samtec" deviceset="CONN-RECEPT-2MM-VERT-AU-10POS" device=""/>
-<part name="U$11" library="samtec" deviceset="CONN-RECEPT-2MM-VERT-AU-10POS" device=""/>
-<part name="U$12" library="samtec" deviceset="CONN-RECEPT-2MM-VERT-AU-10POS" device=""/>
 <part name="PWM" library="NXP" deviceset="PCA9685" device="" value="PCA9685"/>
 <part name="JP1" library="molex" deviceset="2_SUPERSABRE" device="" value="PWR"/>
@@
 <instance part="U$6" gate="G$1" x="-40.64" y="2.54" rot="R270"/>
 <instance part="U$7" gate="G$1" x="-40.64" y="-15.24" rot="R270"/>
-<instance part="U$8" gate="G$1" x="-40.64" y="-30.48" rot="R270"/>
-<instance part="U$9" gate="G$1" x="15.494" y="-30.226" rot="R270"/>
 <instance part="U$10" gate="G$1" x="15.24" y="17.78" rot="R270"/>
-<instance part="U$11" gate="G$1" x="15.24" y="2.54" rot="R270"/>
-<instance part="U$12" gate="G$1" x="15.24" y="-15.24" rot="R270"/>
 <instance part="PWM" gate="G$1" x="58.42" y="38.1"/>
 <instance part="JP1" gate="G$1" x="35.56" y="78.74"/>
@@
 </segment>
 <segment>
-<pinref part="U$3" gate="G$1" pin="2"/>
-<wire x1="71.12" y1="12.7" x2="78.74" y2="12.7" width="0.1524" layer="91"/>
-<label x="73.66" y="12.7" size="1.778" layer="95"/>
-</segment>
-<segment>
-<pinref part="U$3" gate="G$1" pin="3"/>
-<wire x1="71.12" y1="2.54" x2="78.74" y2="2.54" width="0.1524" layer="91"/>
-<label x="73.66" y="2.54" size="1.778" layer="95"/>
-</segment>
-<segment>
-<pinref part="U$4" gate="G$1" pin="2"/>
-<wire x1="71.12" y1="-20.32" x2="81.28" y2="-20.32" width="0.1524" layer="91"/>
-<label x="76.2" y="-20.32" size="1.778" layer="95"/>
-</segment>
-<segment>
-<pinref part="U$4" gate="G$1" pin="3"/>
-<wire x1="71.12" y1="-30.48" x2="81.28" y2="-30.48" width="0.1524" layer="91"/>
-<label x="76.2" y="-30.48" size="1.778" layer="95"/>
-</segment>
-</net>
-<net name="GND" class="0">
-<segment>
 <pinref part="U$1" gate="G$1" pin="2"/>
 <wire x1="-78.74" y1="15.24" x2="-71.12" y2="15.24" width="0.1524" layer="91"/>
 <label x="-76.2" y="15.24" size="1.778" layer="95"/>
-</segment>
-<segment>
-<pinref part="JP1" gate="G$1" pin="P$2"/>
-<wire x1="27.94" y1="76.2" x2="22.86" y2="76.2" width="0.1524" layer="91"/>
-<label x="22.86" y="76.2" size="1.778" layer="95"/>
 </segment>
 <segment>
@@
 <wire x1="-78.74" y1="-30.48" x2="-71.12" y2="-30.48" width="0.1524" layer="91"/>
 <label x="-76.2" y="-30.48" size="1.778" layer="95"/>
+</segment>
+</net>
+<net name="GND" class="0">
+<segment>
+<pinref part="JP1" gate="G$1" pin="P$2"/>
+<wire x1="27.94" y1="76.2" x2="22.86" y2="76.2" width="0.1524" layer="91"/>
+<label x="22.86" y="76.2" size="1.778" layer="95"/>
 </segment>
 <segment>
@@
 <label x="83.82" y="66.04" size="1.778" layer="95"/>
 </segment>
+<segment>
+<pinref part="U$3" gate="G$1" pin="2"/>
+<wire x1="71.12" y1="12.7" x2="78.74" y2="12.7" width="0.1524" layer="91"/>
+<label x="73.66" y="12.7" size="1.778" layer="95"/>
+</segment>
+<segment>
+<pinref part="U$3" gate="G$1" pin="3"/>
+<wire x1="71.12" y1="2.54" x2="78.74" y2="2.54" width="0.1524" layer="91"/>
+<label x="73.66" y="2.54" size="1.778" layer="95"/>
+</segment>
+<segment>
+<pinref part="U$4" gate="G$1" pin="2"/>
+<wire x1="71.12" y1="-20.32" x2="81.28" y2="-20.32" width="0.1524" layer="91"/>
+<label x="76.2" y="-20.32" size="1.778" layer="95"/>
+</segment>
+<segment>
+<pinref part="U$4" gate="G$1" pin="3"/>
+<wire x1="71.12" y1="-30.48" x2="81.28" y2="-30.48" width="0.1524" layer="91"/>
+<label x="76.2" y="-30.48" size="1.778" layer="95"/>
+</segment>
 </net>
