File: Project QUBO/eagleDesigns/Qubo New/BatteryHullBoard/BatteryHullBoard.sch (EAGLE design)
At the start: 8 parts, among them U1 KSK-1E66, U2 CMXSIPSSR

Commit message: Changed Relay on BatteryHubBoard with new one
Parts:
- removed U2: CMXSIPSSR, CMXSIPSSR:CMXSIPSSR
- added U$1: ADJH21112, switch:ADJH21112
Connections:
- net GND: now also U$1.CONTROL-; no longer U2.4
- net N$3: now also U$1.CONTROL+; no longer U2.3
- net PWR1: now also U$1.INPUT; no longer U2.2
- net PWR2: now also U$1.OUTPUT; no longer U2.1
Changed lines of the file:
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@@
 <?xml version="1.0" encoding="utf-8"?>
 <!DOCTYPE eagle SYSTEM "eagle.dtd">
-<eagle version="8.3.2">
+<eagle version="9.2.0">
 <drawing>
 <settings>
@@
 <parts>
 <part name="U1" library="KSK-1E66" deviceset="KSK-1E66" device=""/>
-<part name="U2" library="CMXSIPSSR" deviceset="CMXSIPSSR" device=""/>
 <part name="BATTERY" library="molex" deviceset="2_SUPERSABRE" device=""/>
 <part name="ROBOT" library="molex" deviceset="2_SUPERSABRE" device=""/>
@@
 <part name="FRAME1" library="frames" deviceset="A5L-LOC" device=""/>
 <part name="R3" library="resistor" deviceset="R-US_" device="R0805" value="10000"/>
+<part name="U$1" library="switch" deviceset="ADJH21112" device=""/>
 </parts>
 <sheets>
@@
 </plain>
 <instances>
-<instance part="U1" gate="G$1" x="76.2" y="101.6"/>
-<instance part="U2" gate="G$1" x="114.3" y="101.6"/>
-<instance part="BATTERY" gate="G$1" x="48.26" y="88.9" rot="MR0"/>
-<instance part="ROBOT" gate="G$1" x="124.46" y="78.74"/>
-<instance part="LED1" gate="G$1" x="99.06" y="76.2"/>
-<instance part="R1" gate="G$1" x="81.28" y="83.82" rot="R90"/>
-<instance part="R2" gate="G$1" x="81.28" y="71.12" rot="R90"/>
-<instance part="FRAME1" gate="G$1" x="0" y="0"/>
-<instance part="R3" gate="G$1" x="99.06" y="63.5" rot="R90"/>
+<instance part="U1" gate="G$1" x="76.2" y="101.6">
+<attribute name="NAME" x="66.04" y="96.52" size="1.27" layer="95"/>
+<attribute name="VALUE" x="81.28" y="96.52" size="1.27" layer="96"/>
+</instance>
+<instance part="BATTERY" gate="G$1" x="48.26" y="88.9" rot="MR0">
+<attribute name="VALUE" x="53.34" y="78.74" size="1.778" layer="96" rot="MR0"/>
+<attribute name="NAME" x="53.34" y="96.52" size="1.778" layer="95" rot="MR0"/>
+</instance>
+<instance part="ROBOT" gate="G$1" x="124.46" y="78.74">
+<attribute name="VALUE" x="119.38" y="68.58" size="1.778" layer="96"/>
+<attribute name="NAME" x="119.38" y="86.36" size="1.778" layer="95"/>
+</instance>
+<instance part="LED1" gate="G$1" x="99.06" y="76.2">
+<attribute name="NAME" x="102.616" y="71.628" size="1.778" layer="95" rot="R90"/>
+<attribute name="VALUE" x="104.775" y="71.628" size="1.778" layer="96" rot="R90"/>
+</instance>
+<instance part="R1" gate="G$1" x="81.28" y="83.82" rot="R90">
+<attribute name="NAME" x="79.7814" y="80.01" size="1.778" layer="95" rot="R90"/>
+<attribute name="VALUE" x="84.582" y="80.01" size="1.778" layer="96" rot="R90"/>
+</instance>
+<instance part="R2" gate="G$1" x="81.28" y="71.12" rot="R90">
+<attribute name="NAME" x="79.7814" y="67.31" size="1.778" layer="95" rot="R90"/>
+<attribute name="VALUE" x="84.582" y="67.31" size="1.778" layer="96" rot="R90"/>
+</instance>
+<instance part="FRAME1" gate="G$1" x="0" y="0">
+<attribute name="DRAWING_NAME" x="140.97" y="15.24" size="2.54" layer="94" font="vector"/>
+<attribute name="LAST_DATE_TIME" x="140.97" y="10.16" size="2.286" layer="94" font="vector"/>
+<attribute name="SHEET" x="154.305" y="5.08" size="2.54" layer="94" font="vector"/>
+</instance>
+<instance part="R3" gate="G$1" x="99.06" y="63.5" rot="R90">
+<attribute name="NAME" x="97.5614" y="59.69" size="1.778" layer="95" rot="R90"/>
+<attribute name="VALUE" x="102.362" y="59.69" size="1.778" layer="96" rot="R90"/>
+</instance>
+<instance part="U$1" gate="G$1" x="129.54" y="104.14" rot="MR0"/>
 </instances>
 <busses>
@@
 <wire x1="60.96" y1="101.6" x2="60.96" y2="109.22" width="0.1524" layer="91"/>
 <junction x="60.96" y="101.6"/>
-<wire x1="101.6" y1="109.22" x2="101.6" y2="88.9" width="0.1524" layer="91"/>
-<pinref part="U2" gate="G$1" pin="2"/>
-<wire x1="101.6" y1="88.9" x2="111.76" y2="88.9" width="0.1524" layer="91"/>
-<wire x1="111.76" y1="88.9" x2="111.76" y2="93.98" width="0.1524" layer="91"/>
-<wire x1="60.96" y1="109.22" x2="101.6" y2="109.22" width="0.1524" layer="91"/>
+<wire x1="60.96" y1="109.22" x2="105.04" y2="109.22" width="0.1524" layer="91"/>
 <label x="60.96" y="91.44" size="1.778" layer="95"/>
+<pinref part="U$1" gate="G$1" pin="INPUT"/>
+<wire x1="105.04" y1="109.22" x2="105.04" y2="108.14" width="0.1524" layer="91"/>
 </segment>
 </net>
@@
 </segment>
 <segment>
-<pinref part="U2" gate="G$1" pin="4"/>
-<wire x1="121.92" y1="93.98" x2="127" y2="93.98" width="0.1524" layer="91"/>
-<label x="124.46" y="93.98" size="1.778" layer="95"/>
+<wire x1="165.1" y1="109.22" x2="170.18" y2="109.22" width="0.1524" layer="91"/>
+<label x="165.1" y="111.76" size="1.778" layer="95"/>
+<pinref part="U$1" gate="G$1" pin="CONTROL-"/>
+<wire x1="154.04" y1="108.14" x2="165.1" y2="108.14" width="0.1524" layer="91"/>
+<wire x1="165.1" y1="108.14" x2="165.1" y2="109.22" width="0.1524" layer="91"/>
 </segment>
 </net>
@@
 <junction x="81.28" y="78.74"/>
 <wire x1="114.3" y1="78.74" x2="114.3" y2="88.9" width="0.1524" layer="91"/>
-<pinref part="U2" gate="G$1" pin="3"/>
 <wire x1="114.3" y1="88.9" x2="116.84" y2="88.9" width="0.1524" layer="91"/>
 <wire x1="116.84" y1="88.9" x2="116.84" y2="93.98" width="0.1524" layer="91"/>
 <wire x1="99.06" y1="78.74" x2="114.3" y2="78.74" width="0.1524" layer="91"/>
 <junction x="99.06" y="78.74"/>
+<pinref part="U$1" gate="G$1" pin="CONTROL+"/>
+<wire x1="116.84" y1="93.98" x2="154.04" y2="93.98" width="0.1524" layer="91"/>
+<wire x1="154.04" y1="93.98" x2="154.04" y2="101.14" width="0.1524" layer="91"/>
 </segment>
 </net>
 <net name="PWR2" class="0">
 <segment>
-<pinref part="U2" gate="G$1" pin="1"/>
 <wire x1="106.68" y1="93.98" x2="106.68" y2="83.82" width="0.1524" layer="91"/>
 <pinref part="ROBOT" gate="G$1" pin="P$1"/>
 <wire x1="106.68" y1="83.82" x2="116.84" y2="83.82" width="0.1524" layer="91"/>
 <wire x1="116.84" y1="83.82" x2="116.84" y2="81.28" width="0.1524" layer="91"/>
-</segment>
-</net>
+<pinref part="U$1" gate="G$1" pin="OUTPUT"/>
+<wire x1="106.68" y1="93.98" x2="105.04" y2="93.98" width="0.1524" layer="91"/>
+<wire x1="105.04" y1="93.98" x2="105.04" y2="101.14" width="0.1524" layer="91"/>
+</segment>
+</net>
