File: Project_QUBO/eagleDesigns/Qubo_New/Power Board/Powerboard.brd (EAGLE design)
At the start: 127 x 88.9 mm, 34 parts, among them IC1 PCF8574T, U1 UEI15, U2 TSR2-2450

Commit message: created HyperArmboard
Parts:
- moved C6 135.5 mm to (113.0, 23.9), turned to 90 degrees
- moved C5 79.3 mm to (60.2, 26.2)
- renumbered IC1 to IO-EXPANDER, U$2 to A-2-D
Connections:
- removed net 5V_EN: IO-EXPANDER.5
- removed net UEI_INPUT: U1.P$5, UWE_CURRENT_SENSOR.P$3, UWE_CURRENT_SENSOR.P$4
- new net N$6: U1.+VIN, UWE_CURRENT_SENSOR.P$3, UWE_CURRENT_SENSOR.P$4
- net GND: now also U1.-VIN; no longer U1.P$6
- net PROCESSED_UEI_OUTPUT: now also U1.+VOUT; no longer U1.P$1
- net UEI_EN: now also U1.ON/OFFCNTRL; no longer U1.P$4
- net UEI_GND: now also U1.-VOUT; no longer U1.P$3
Routing:
- net 10V_OUT: track 9.97 -> 19.0 mm
- net PROCESSED_INPUT: track 93.3 -> 101.8 mm
- net GND: track 86.1 -> 79.2 mm
- net N$6: track 0.00 -> 1.27 mm
- net UEI_EN: track 75.4 -> 74.9 mm
- net PROCESSED_10V_OUT: track 116.5 -> 116.3 mm, vias 4 -> 2
- added copper zone on layer 1, net N$6
- removed copper zone on layer 1, net UEI_INPUT
